File: schematics/DualCore6502Whole/DualCore6502Whole.kicad_sch (KiCad schematic)
At the start: 17 parts, among them J1 VIN, J2 PWR, SW1 Power, SW2 RESET, U1 LM7805

Commit message: Update the schematic
Other:
- title: (none) -> Dual Core 65C02 Computer
Changed lines of the file:
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@@
 	(generator_version "8.0")
 	(paper "A4")
+	(title_block
+		(title "Dual Core 65C02 Computer")
+		(date "2026")
+		(comment 1 "Copyright (c) 2026 Rhys Weatherley")
+		(comment 3 "Power Supply and Reset")
+	)
 	(junction
 		(at 86.36 104.14)

Commit message: Update schematic and add 1ms NMI tick
Other:
- added sheet Tick Timer (tick_timer.kicad_sch)
Changed lines of the file:
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@@
+	)
+	(sheet
+		(at 192.278 48.006)
+		(size 34.544 16.256)
+		(fields_autoplaced yes)
+		(stroke
+			(width 0.1524)
+			(type solid)
+		)
+		(fill
+			(color 0 0 0 0.0000)
+		)
+		(property "Sheetname" "Tick Timer"
+			(at 192.278 47.2944 0)
+			(effects
+				(font
+					(size 1.27 1.27)
+				)
+				(justify left bottom)
+			)
+		)
+		(property "Sheetfile" "tick_timer.kicad_sch"
+			(at 192.278 64.8466 0)
+			(effects
+				(font
+					(size 1.27 1.27)
+				)
+				(justify left top)
+			)
+		)
+		(instances
+			(project "DualCore6502Whole"
+				(path "/93e0914e-b2e9-49c2-95f2-7cc419f4ea20"
+					(page "11")
+				)
+			)
+		)
 	)
 	(sheet

Commit message: Basic PCB layout
Parts:
- removed C2: 100nF, Capacitor_THT:C_Disc_D5.0mm_W2.5mm_P5.00mm, symbol Device:C
- removed D1: 1N5819, Diode_THT:D_DO-41_SOD81_P10.16mm_Horizontal, symbol Diode:1N5819
- removed J2: PWR, Connector_PinHeader_2.54mm:PinHeader_1x04_P2.54mm_Vertical, symbol Connector_Generic:Conn_01x04
- removed U1: LM7805, Package_TO_SOT_THT:TO-220-3_Horizontal_TabDown, symbol Regulator_Linear:L7805
- added J2: PWR, Connector_Phoenix_MC_HighVoltage:PhoenixContact_MC_1,5_3-G-5.08_1x03_P5.08mm_Horizontal, symbol Connector_Generic:Conn_01x03
- C1: value 47uF -> 100uF
- D1: renamed from D2; value Power On -> Power
- J1: value VIN -> 5VDC
- R1: value 220R -> 470R
- SW1: value Power -> Power On
- renumbered C3 to C2
Connections:
- net VDD is gone; now on net +5V: SW1.1 (A)
- net +5V: now also C1.1, J2.1 (Pin_1)
- net GND: now also J2.3 (Pin_3)
- net ~{RESET}: now also J2.2 (Pin_2)
Other:
- note added: "For supplying 5V from off-board, or for supplying 5V to off-board."
- note removed: "9VDC to 12VDC"
- moved on the sheet: C1, D1, R1
