File: schematics/DualCore6502Whole/acia.kicad_sch (KiCad schematic)
At the start: 12 parts, among them J4 RS232, U16 W65C51N, U17 MAX232, Y2 1.8432MHz

Commit message: Remove the need to multiplex the control lines
Parts:
- renumbered C18 to C17, C19 to C18, C20 to C19, C21 to C20, C22 to C21, C23 to C22, U16 to U15, U17 to U16
Changed lines of the file:
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@@
 		(dnp no)
 		(fields_autoplaced yes)
-		(property "Reference" "U17"
+		(property "Reference" "U16"
 			(at 196.5041 67.31 0)
 			(effects
@@
 			(project "DualCore6502Whole"
 				(path "/93e0914e-b2e9-49c2-95f2-7cc419f4ea20/659d2ec5-e43d-4409-be3e-c470dc127456"
-					(reference "U17")
+					(reference "U16")
 					(unit 1)
 				)
@@
 		(dnp no)
 		(fields_autoplaced yes)
-		(property "Reference" "U16"
+		(property "Reference" "U15"
 			(at 96.1741 60.96 0)
 			(effects
@@
 			(project ""
 				(path "/93e0914e-b2e9-49c2-95f2-7cc419f4ea20/659d2ec5-e43d-4409-be3e-c470dc127456"
-					(reference "U16")
+					(reference "U15")
 					(unit 1)
 				)
@@
 		(dnp no)
 		(fields_autoplaced yes)
-		(property "Reference" "C20"
+		(property "Reference" "C19"
 			(at 168.91 77.47 0)
 			(effects
@@
 			(project "DualCore6502Whole"
 				(path "/93e0914e-b2e9-49c2-95f2-7cc419f4ea20/659d2ec5-e43d-4409-be3e-c470dc127456"
-					(reference "C20")
+					(reference "C19")
 					(unit 1)
 				)
@@
 		(dnp no)
 		(fields_autoplaced yes)
-		(property "Reference" "C23"
+		(property "Reference" "C22"
 			(at 238.76 123.19 0)
 			(effects
@@
 			(project "DualCore6502Whole"
 				(path "/93e0914e-b2e9-49c2-95f2-7cc419f4ea20/659d2ec5-e43d-4409-be3e-c470dc127456"
-					(reference "C23")
+					(reference "C22")
 					(unit 1)
 				)
@@
 		(dnp no)
 		(fields_autoplaced yes)
-		(property "Reference" "#PWR96"
+		(property "Reference" "#PWR89"
 			(at 115.57 124.46 0)
 			(effects
@@
 			(project "DualCore6502Whole"
 				(path "/93e0914e-b2e9-49c2-95f2-7cc419f4ea20/659d2ec5-e43d-4409-be3e-c470dc127456"
-					(reference "#PWR96")
+					(reference "#PWR89")
 					(unit 1)
 				)
@@
 		(dnp no)
 		(fields_autoplaced yes)
-		(property "Reference" "#PWR93"
+		(property "Reference" "#PWR86"
 			(at 19.05 101.6 0)
 			(effects
@@
 			(project "DualCore6502Whole"
 				(path "/93e0914e-b2e9-49c2-95f2-7cc419f4ea20/659d2ec5-e43d-4409-be3e-c470dc127456"
-					(reference "#PWR93")
+					(reference "#PWR86")
 					(unit 1)
 				)
@@
 		(dnp no)
 		(fields_autoplaced yes)
-		(property "Reference" "#PWR97"
+		(property "Reference" "#PWR90"
 			(at 149.86 81.28 0)
 			(effects
@@
 			(project "DualCore6502Whole"
 				(path "/93e0914e-b2e9-49c2-95f2-7cc419f4ea20/659d2ec5-e43d-4409-be3e-c470dc127456"
-					(reference "#PWR97")
+					(reference "#PWR90")
 					(unit 1)
 				)
@@
 		(dnp no)
 		(fields_autoplaced yes)
-		(property "Reference" "C21"
+		(property "Reference" "C20"
 			(at 227.33 123.19 0)
 			(effects
@@
 			(project "DualCore6502Whole"
 				(path "/93e0914e-b2e9-49c2-95f2-7cc419f4ea20/659d2ec5-e43d-4409-be3e-c470dc127456"
-					(reference "C21")
+					(reference "C20")
 					(unit 1)
 				)
@@
 		(dnp no)
 		(fields_autoplaced yes)
-		(property "Reference" "#PWR92"
+		(property "Reference" "#PWR85"
 			(at 19.05 91.44 0)
 			(effects
@@
 			(project ""
 				(path "/93e0914e-b2e9-49c2-95f2-7cc419f4ea20/659d2ec5-e43d-4409-be3e-c470dc127456"
-					(reference "#PWR92")
+					(reference "#PWR85")
 					(unit 1)
 				)
@@
 		(dnp no)
 		(fields_autoplaced yes)
-		(property "Reference" "C18"
+		(property "Reference" "C17"
 			(at 22.86 90.17 0)
 			(effects
@@
 			(project "DualCore6502Whole"
 				(path "/93e0914e-b2e9-49c2-95f2-7cc419f4ea20/659d2ec5-e43d-4409-be3e-c470dc127456"
-					(reference "C18")
+					(reference "C17")
 					(unit 1)
 				)
@@
 		(dnp no)
 		(fields_autoplaced yes)
-		(property "Reference" "#PWR99"
+		(property "Reference" "#PWR92"
 			(at 194.31 134.62 0)
 			(effects
@@
 			(project "DualCore6502Whole"
 				(path "/93e0914e-b2e9-49c2-95f2-7cc419f4ea20/659d2ec5-e43d-4409-be3e-c470dc127456"
-					(reference "#PWR99")
+					(reference "#PWR92")
 					(unit 1)
 				)
@@
 		(dnp no)
 		(fields_autoplaced yes)
-		(property "Reference" "#PWR102"
+		(property "Reference" "#PWR95"
 			(at 256.54 124.46 0)
 			(effects
@@
 			(project "DualCore6502Whole"
 				(path "/93e0914e-b2e9-49c2-95f2-7cc419f4ea20/659d2ec5-e43d-4409-be3e-c470dc127456"
-					(reference "#PWR102")
+					(reference "#PWR95")
 					(unit 1)
 				)
@@
 		(dnp no)
 		(fields_autoplaced yes)
-		(property "Reference" "#PWR101"
+		(property "Reference" "#PWR94"
 			(at 234.95 134.62 0)
 			(effects
@@
 			(project "DualCore6502Whole"
 				(path "/93e0914e-b2e9-49c2-95f2-7cc419f4ea20/659d2ec5-e43d-4409-be3e-c470dc127456"
-					(reference "#PWR101")
+					(reference "#PWR94")
 					(unit 1)
 				)
@@
 		(dnp no)
 		(fields_autoplaced yes)
-		(property "Reference" "#PWR98"
+		(property "Reference" "#PWR91"
 			(at 194.31 71.12 0)
 			(effects
@@
 			(project "DualCore6502Whole"
 				(path "/93e0914e-b2e9-49c2-95f2-7cc419f4ea20/659d2ec5-e43d-4409-be3e-c470dc127456"
-					(reference "#PWR98")
+					(reference "#PWR91")
 					(unit 1)
 				)
@@
 		(dnp no)
 		(fields_autoplaced yes)
-		(property "Reference" "#PWR95"
+		(property "Reference" "#PWR88"
 			(at 93.98 140.97 0)
 			(effects
@@
 			(project ""
 				(path "/93e0914e-b2e9-49c2-95f2-7cc419f4ea20/659d2ec5-e43d-4409-be3e-c470dc127456"
-					(reference "#PWR95")
+					(reference "#PWR88")
 					(unit 1)
 				)
@@
 		(dnp no)
 		(fields_autoplaced yes)
-		(property "Reference" "C22"
+		(property "Reference" "C21"
 			(at 228.6 77.47 0)
 			(effects
@@
 			(project "DualCore6502Whole"
 				(path "/93e0914e-b2e9-49c2-95f2-7cc419f4ea20/659d2ec5-e43d-4409-be3e-c470dc127456"
-					(reference "C22")
+					(reference "C21")
 					(unit 1)
 				)
@@
 		(dnp no)
 		(fields_autoplaced yes)
-		(property "Reference" "#PWR100"
+		(property "Reference" "#PWR93"
 			(at 223.52 134.62 0)
 			(effects
@@
 			(project "DualCore6502Whole"
 				(path "/93e0914e-b2e9-49c2-95f2-7cc419f4ea20/659d2ec5-e43d-4409-be3e-c470dc127456"
-					(reference "#PWR100")
+					(reference "#PWR93")
 					(unit 1)
 				)
@@
 		(dnp no)
 		(fields_autoplaced yes)
-		(property "Reference" "#PWR94"
+		(property "Reference" "#PWR87"
 			(at 93.98 64.77 0)
 			(effects
@@
 			(project "DualCore6502Whole"
 				(path "/93e0914e-b2e9-49c2-95f2-7cc419f4ea20/659d2ec5-e43d-4409-be3e-c470dc127456"
-					(reference "#PWR94")
+					(reference "#PWR87")
 					(unit 1)
 				)
@@
 		(dnp no)
 		(fields_autoplaced yes)
-		(property "Reference" "C19"
+		(property "Reference" "C18"
 			(at 153.67 69.85 0)
 			(effects
@@
 			(project "DualCore6502Whole"
 				(path "/93e0914e-b2e9-49c2-95f2-7cc419f4ea20/659d2ec5-e43d-4409-be3e-c470dc127456"
-					(reference "C19")
-					(unit 1)
-				)
+					(reference "C18")
+					(unit 1)
+				)

Commit message: Add simpler I/O outputs as an alternative to the VIA
Parts:
- renumbered C17 to C19, C18 to C20, C19 to C21, C20 to C22, C21 to C23, C22 to C24, J4 to J5, U15 to U17, U16 to U18
Changed lines of the file:
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@@
 		(dnp no)
 		(fields_autoplaced yes)
-		(property "Reference" "U16"
+		(property "Reference" "U18"
 			(at 196.5041 67.31 0)
 			(effects
@@
 			(project "DualCore6502Whole"
 				(path "/93e0914e-b2e9-49c2-95f2-7cc419f4ea20/659d2ec5-e43d-4409-be3e-c470dc127456"
-					(reference "U16")
+					(reference "U18")
 					(unit 1)
 				)
@@
 		(dnp no)
 		(fields_autoplaced yes)
-		(property "Reference" "U15"
+		(property "Reference" "U17"
 			(at 96.1741 60.96 0)
 			(effects
@@
 			(project ""
 				(path "/93e0914e-b2e9-49c2-95f2-7cc419f4ea20/659d2ec5-e43d-4409-be3e-c470dc127456"
-					(reference "U15")
+					(reference "U17")
 					(unit 1)
 				)
@@
 		(dnp no)
 		(fields_autoplaced yes)
-		(property "Reference" "C19"
+		(property "Reference" "C21"
 			(at 168.91 77.47 0)
 			(effects
@@
 			(project "DualCore6502Whole"
 				(path "/93e0914e-b2e9-49c2-95f2-7cc419f4ea20/659d2ec5-e43d-4409-be3e-c470dc127456"
-					(reference "C19")
+					(reference "C21")
 					(unit 1)
 				)
@@
 		(dnp no)
 		(fields_autoplaced yes)
-		(property "Reference" "C22"
+		(property "Reference" "C24"
 			(at 238.76 123.19 0)
 			(effects
@@
 			(project "DualCore6502Whole"
 				(path "/93e0914e-b2e9-49c2-95f2-7cc419f4ea20/659d2ec5-e43d-4409-be3e-c470dc127456"
-					(reference "C22")
+					(reference "C24")
 					(unit 1)
 				)
@@
 		(dnp no)
 		(fields_autoplaced yes)
-		(property "Reference" "#PWR89"
+		(property "Reference" "#PWR99"
 			(at 115.57 124.46 0)
 			(effects
@@
 			(project "DualCore6502Whole"
 				(path "/93e0914e-b2e9-49c2-95f2-7cc419f4ea20/659d2ec5-e43d-4409-be3e-c470dc127456"
-					(reference "#PWR89")
+					(reference "#PWR99")
 					(unit 1)
 				)
@@
 		(dnp no)
 		(fields_autoplaced yes)
-		(property "Reference" "#PWR86"
+		(property "Reference" "#PWR96"
 			(at 19.05 101.6 0)
 			(effects
@@
 			(project "DualCore6502Whole"
 				(path "/93e0914e-b2e9-49c2-95f2-7cc419f4ea20/659d2ec5-e43d-4409-be3e-c470dc127456"
-					(reference "#PWR86")
+					(reference "#PWR96")
 					(unit 1)
 				)
@@
 		(dnp no)
 		(fields_autoplaced yes)
-		(property "Reference" "#PWR90"
+		(property "Reference" "#PWR100"
 			(at 149.86 81.28 0)
 			(effects
@@
 			(project "DualCore6502Whole"
 				(path "/93e0914e-b2e9-49c2-95f2-7cc419f4ea20/659d2ec5-e43d-4409-be3e-c470dc127456"
-					(reference "#PWR90")
+					(reference "#PWR100")
 					(unit 1)
 				)
@@
 		(dnp no)
 		(fields_autoplaced yes)
-		(property "Reference" "J4"
+		(property "Reference" "J5"
 			(at 271.78 104.1399 0)
 			(effects
@@
 			(project "DualCore6502Whole"
 				(path "/93e0914e-b2e9-49c2-95f2-7cc419f4ea20/659d2ec5-e43d-4409-be3e-c470dc127456"
-					(reference "J4")
+					(reference "J5")
 					(unit 1)
 				)
@@
 		(dnp no)
 		(fields_autoplaced yes)
-		(property "Reference" "C20"
+		(property "Reference" "C22"
 			(at 227.33 123.19 0)
 			(effects
@@
 			(project "DualCore6502Whole"
 				(path "/93e0914e-b2e9-49c2-95f2-7cc419f4ea20/659d2ec5-e43d-4409-be3e-c470dc127456"
-					(reference "C20")
+					(reference "C22")
 					(unit 1)
 				)
@@
 		(dnp no)
 		(fields_autoplaced yes)
-		(property "Reference" "#PWR85"
+		(property "Reference" "#PWR95"
 			(at 19.05 91.44 0)
 			(effects
@@
 			(project ""
 				(path "/93e0914e-b2e9-49c2-95f2-7cc419f4ea20/659d2ec5-e43d-4409-be3e-c470dc127456"
-					(reference "#PWR85")
+					(reference "#PWR95")
 					(unit 1)
 				)
@@
 		(dnp no)
 		(fields_autoplaced yes)
-		(property "Reference" "C17"
+		(property "Reference" "C19"
 			(at 22.86 90.17 0)
 			(effects
@@
 			(project "DualCore6502Whole"
 				(path "/93e0914e-b2e9-49c2-95f2-7cc419f4ea20/659d2ec5-e43d-4409-be3e-c470dc127456"
-					(reference "C17")
+					(reference "C19")
 					(unit 1)
 				)
@@
 		(dnp no)
 		(fields_autoplaced yes)
-		(property "Reference" "#PWR92"
+		(property "Reference" "#PWR102"
 			(at 194.31 134.62 0)
 			(effects
@@
 			(project "DualCore6502Whole"
 				(path "/93e0914e-b2e9-49c2-95f2-7cc419f4ea20/659d2ec5-e43d-4409-be3e-c470dc127456"
-					(reference "#PWR92")
+					(reference "#PWR102")
 					(unit 1)
 				)
@@
 		(dnp no)
 		(fields_autoplaced yes)
-		(property "Reference" "#PWR95"
+		(property "Reference" "#PWR105"
 			(at 256.54 124.46 0)
 			(effects
@@
 			(project "DualCore6502Whole"
 				(path "/93e0914e-b2e9-49c2-95f2-7cc419f4ea20/659d2ec5-e43d-4409-be3e-c470dc127456"
-					(reference "#PWR95")
+					(reference "#PWR105")
 					(unit 1)
 				)
@@
 		(dnp no)
 		(fields_autoplaced yes)
-		(property "Reference" "#PWR94"
+		(property "Reference" "#PWR104"
 			(at 234.95 134.62 0)
 			(effects
@@
 			(project "DualCore6502Whole"
 				(path "/93e0914e-b2e9-49c2-95f2-7cc419f4ea20/659d2ec5-e43d-4409-be3e-c470dc127456"
-					(reference "#PWR94")
+					(reference "#PWR104")
 					(unit 1)
 				)
@@
 		(dnp no)
 		(fields_autoplaced yes)
-		(property "Reference" "#PWR91"
+		(property "Reference" "#PWR101"
 			(at 194.31 71.12 0)
 			(effects
@@
 			(project "DualCore6502Whole"
 				(path "/93e0914e-b2e9-49c2-95f2-7cc419f4ea20/659d2ec5-e43d-4409-be3e-c470dc127456"
-					(reference "#PWR91")
+					(reference "#PWR101")
 					(unit 1)
 				)
@@
 		(dnp no)
 		(fields_autoplaced yes)
-		(property "Reference" "#PWR88"
+		(property "Reference" "#PWR98"
 			(at 93.98 140.97 0)
 			(effects
@@
 			(project ""
 				(path "/93e0914e-b2e9-49c2-95f2-7cc419f4ea20/659d2ec5-e43d-4409-be3e-c470dc127456"
-					(reference "#PWR88")
+					(reference "#PWR98")
 					(unit 1)
 				)
@@
 		(dnp no)
 		(fields_autoplaced yes)
-		(property "Reference" "C21"
+		(property "Reference" "C23"
 			(at 228.6 77.47 0)
 			(effects
@@
 			(project "DualCore6502Whole"
 				(path "/93e0914e-b2e9-49c2-95f2-7cc419f4ea20/659d2ec5-e43d-4409-be3e-c470dc127456"
-					(reference "C21")
+					(reference "C23")
 					(unit 1)
 				)
@@
 		(dnp no)
 		(fields_autoplaced yes)
-		(property "Reference" "#PWR93"
+		(property "Reference" "#PWR103"
 			(at 223.52 134.62 0)
 			(effects
@@
 			(project "DualCore6502Whole"
 				(path "/93e0914e-b2e9-49c2-95f2-7cc419f4ea20/659d2ec5-e43d-4409-be3e-c470dc127456"
-					(reference "#PWR93")
+					(reference "#PWR103")
 					(unit 1)
 				)
@@
 		(dnp no)
 		(fields_autoplaced yes)
-		(property "Reference" "#PWR87"
+		(property "Reference" "#PWR97"
 			(at 93.98 64.77 0)
 			(effects
@@
 			(project "DualCore6502Whole"
 				(path "/93e0914e-b2e9-49c2-95f2-7cc419f4ea20/659d2ec5-e43d-4409-be3e-c470dc127456"
-					(reference "#PWR87")
+					(reference "#PWR97")
 					(unit 1)
 				)
@@
 		(dnp no)
 		(fields_autoplaced yes)
-		(property "Reference" "C18"
+		(property "Reference" "C20"
 			(at 153.67 69.85 0)
 			(effects
@@
 			(project "DualCore6502Whole"
 				(path "/93e0914e-b2e9-49c2-95f2-7cc419f4ea20/659d2ec5-e43d-4409-be3e-c470dc127456"
-					(reference "C18")
-					(unit 1)
-				)
+					(reference "C20")
+					(unit 1)
+				)

Commit message: Update the schematic
Parts:
- added JP2: ACIA IRQ, Connector_PinHeader_2.54mm:PinHeader_1x03_P2.54mm_Vertical, symbol Jumper:Jumper_3_Bridged12
- renumbered C19 to C22, C20 to C23, C21 to C24, C22 to C25, C23 to C26, C24 to C27, D4 to D9, R9 to R14, U17 to U20, U18 to U21
Connections:
- net ~{CPU2_IRQ}: now also JP2.3 (B); no longer D9.2 (A)
- net at U20.8 (~{RTS}): no longer U21.10 (T2IN)
- net at U21.8 (R2IN): now also J5.7
- net ~{CTS}: now reaches U21.9 (R2OUT)
- net CPU2_CLK renamed COMMON_CLK
- new net: D9.2 (A), JP2.2 (C)
- new net ~{CPU1_IRQ}: JP2.1 (A)
- new net ~{RTS}: U21.10 (T2IN)
- no-connect marks 10 -> 8
Other:
- note added: "W65C51N has a bug where ~{RTS} doesn't work properly. Instead, ~{RTS} is controlled by a GPIO."
- title: (none) -> Dual Core 65C02 Computer
- moved on the sheet: C22, D9

Commit message: Update schematic and add 1ms NMI tick
Parts:
- removed JP2: ACIA IRQ, Connector_PinHeader_2.54mm:PinHeader_1x03_P2.54mm_Vertical, symbol Jumper:Jumper_3_Bridged12
Connections:
- net ~{CPU1_IRQ}: now also D9.2 (A)
Changed lines of the file:
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@@
-	(wire
-		(pts
-			(xy 43.18 66.04) (xy 43.18 71.12)
-		)
-		(stroke
-			(width 0)
-			(type default)
-		)
-	)
 	(wire
 		(pts
@@
 	(wire
 		(pts
-			(xy 38.1 88.9) (xy 43.18 88.9)
-		)
-		(stroke
-			(width 0)
-			(type default)
-		)
-	)
-	(wire
-		(pts
 			(xy 109.22 107.95) (xy 115.57 107.95)
 		)
@@
 		)
 	)
-	(wire
-		(pts
-			(xy 43.18 88.9) (xy 43.18 83.82)
-		)
-		(stroke
-			(width 0)
-			(type default)
-		)
-	)
 	(bus
 		(pts
@@
 		(pts
 			(xy 243.84 115.57) (xy 214.63 115.57)
-		)
-		(stroke
-			(width 0)
-			(type default)
-		)
-	)
-	(wire
-		(pts
-			(xy 38.1 66.04) (xy 43.18 66.04)
 		)
 		(stroke
@@
 	(global_label "~{CPU1_IRQ}"
 		(shape output)
-		(at 38.1 66.04 180)
+		(at 46.99 77.47 180)
 		(fields_autoplaced yes)
 		(effects
@@
 		)
 		(property "Intersheetrefs" "${INTERSHEET_REFS}"
-			(at 25.8619 66.04 0)
-			(effects
-				(font
-					(size 1.27 1.27)
-				)
-				(justify right)
-				(hide yes)
-			)
-		)
-	)
-	(global_label "~{CPU2_IRQ}"
-		(shape output)
-		(at 38.1 88.9 180)
-		(fields_autoplaced yes)
-		(effects
-			(font
-				(size 1.27 1.27)
-			)
-			(justify right)
-		)
-		(property "Intersheetrefs" "${INTERSHEET_REFS}"
-			(at 25.8619 88.9 0)
+			(at 34.7519 77.47 0)
 			(effects
 				(font
@@
 		(dnp no)
 		(fields_autoplaced yes)
-		(property "Reference" "#PWR127"
+		(property "Reference" "#PWR126"
 			(at 115.57 124.46 0)
 			(effects
@@
 			(project "DualCore6502Whole"
 				(path "/93e0914e-b2e9-49c2-95f2-7cc419f4ea20/659d2ec5-e43d-4409-be3e-c470dc127456"
-					(reference "#PWR127")
+					(reference "#PWR126")
 					(unit 1)
 				)
@@
 		(dnp no)
 		(fields_autoplaced yes)
-		(property "Reference" "#PWR124"
+		(property "Reference" "#PWR123"
 			(at 73.66 59.69 0)
 			(effects
@@
 			(project "DualCore6502Whole"
 				(path "/93e0914e-b2e9-49c2-95f2-7cc419f4ea20/659d2ec5-e43d-4409-be3e-c470dc127456"
-					(reference "#PWR124")
+					(reference "#PWR123")
 					(unit 1)
 				)
@@
 		(dnp no)
 		(fields_autoplaced yes)
-		(property "Reference" "#PWR128"
+		(property "Reference" "#PWR127"
 			(at 149.86 81.28 0)
 			(effects
@@
 			(project "DualCore6502Whole"
 				(path "/93e0914e-b2e9-49c2-95f2-7cc419f4ea20/659d2ec5-e43d-4409-be3e-c470dc127456"
-					(reference "#PWR128")
-					(unit 1)
-				)
-			)
-		)
-	)
-	(symbol
-		(lib_id "Jumper:Jumper_3_Bridged12")
-		(at 43.18 77.47 90)
-		(mirror x)
-		(unit 1)
-		(exclude_from_sim yes)
-		(in_bom no)
-		(on_board yes)
-		(dnp no)
-		(fields_autoplaced yes)
-		(property "Reference" "JP2"
-			(at 40.64 76.1999 90)
-			(effects
-				(font
-					(size 1.27 1.27)
-				)
-				(justify left)
-			)
-		)
-		(property "Value" "ACIA IRQ"
-			(at 40.64 78.7399 90)
-			(effects
-				(font
-					(size 1.27 1.27)
-				)
-				(justify left)
-			)
-		)
-		(property "Footprint" "Connector_PinHeader_2.54mm:PinHeader_1x03_P2.54mm_Vertical"
-			(at 43.18 77.47 0)
-			(effects
-				(font
-					(size 1.27 1.27)
-				)
-				(hide yes)
-			)
-		)
-		(property "Datasheet" "~"
-			(at 43.18 77.47 0)
-			(effects
-				(font
-					(size 1.27 1.27)
-				)
-				(hide yes)
-			)
-		)
-		(property "Description" "Jumper, 3-pole, pins 1+2 closed/bridged"
-			(at 43.18 77.47 0)
-			(effects
-				(font
-					(size 1.27 1.27)
-				)
-				(hide yes)
-			)
-		)
-		(pin "3"
-		)
-		(pin "2"
-		)
-		(pin "1"
-		)
-		(instances
-			(project "DualCore6502Whole"
-				(path "/93e0914e-b2e9-49c2-95f2-7cc419f4ea20/659d2ec5-e43d-4409-be3e-c470dc127456"
-					(reference "JP2")
+					(reference "#PWR127")
 					(unit 1)
 				)
@@
 		(dnp no)
 		(fields_autoplaced yes)
-		(property "Reference" "#PWR123"
+		(property "Reference" "#PWR122"
 			(at 73.66 49.53 0)
 			(effects
@@
 			(project ""
 				(path "/93e0914e-b2e9-49c2-95f2-7cc419f4ea20/659d2ec5-e43d-4409-be3e-c470dc127456"
-					(reference "#PWR123")
+					(reference "#PWR122")
 					(unit 1)
 				)
@@
 		(dnp no)
 		(fields_autoplaced yes)
-		(property "Reference" "#PWR130"
+		(property "Reference" "#PWR129"
 			(at 194.31 134.62 0)
 			(effects
@@
 			(project "DualCore6502Whole"
 				(path "/93e0914e-b2e9-49c2-95f2-7cc419f4ea20/659d2ec5-e43d-4409-be3e-c470dc127456"
-					(reference "#PWR130")
+					(reference "#PWR129")
 					(unit 1)
 				)
@@
 		(dnp no)
 		(fields_autoplaced yes)
-		(property "Reference" "#PWR133"
+		(property "Reference" "#PWR132"
 			(at 256.54 124.46 0)
 			(effects
@@
 			(project "DualCore6502Whole"
 				(path "/93e0914e-b2e9-49c2-95f2-7cc419f4ea20/659d2ec5-e43d-4409-be3e-c470dc127456"
-					(reference "#PWR133")
+					(reference "#PWR132")
 					(unit 1)
 				)
@@
 		(dnp no)
 		(fields_autoplaced yes)
-		(property "Reference" "#PWR132"
+		(property "Reference" "#PWR131"
 			(at 234.95 134.62 0)
 			(effects
@@
 			(project "DualCore6502Whole"
 				(path "/93e0914e-b2e9-49c2-95f2-7cc419f4ea20/659d2ec5-e43d-4409-be3e-c470dc127456"
-					(reference "#PWR132")
+					(reference "#PWR131")
 					(unit 1)
 				)
@@
 		(dnp no)
 		(fields_autoplaced yes)
-		(property "Reference" "#PWR129"
+		(property "Reference" "#PWR128"
 			(at 194.31 71.12 0)
 			(effects
@@
 			(project "DualCore6502Whole"
 				(path "/93e0914e-b2e9-49c2-95f2-7cc419f4ea20/659d2ec5-e43d-4409-be3e-c470dc127456"
-					(reference "#PWR129")
+					(reference "#PWR128")
 					(unit 1)
 				)
@@
 		(dnp no)
 		(fields_autoplaced yes)
-		(property "Reference" "#PWR126"
+		(property "Reference" "#PWR125"
 			(at 93.98 140.97 0)
 			(effects
@@
 			(project ""
 				(path "/93e0914e-b2e9-49c2-95f2-7cc419f4ea20/659d2ec5-e43d-4409-be3e-c470dc127456"
-					(reference "#PWR126")
+					(reference "#PWR125")
 					(unit 1)
 				)
@@
 		(dnp no)
 		(fields_autoplaced yes)
-		(property "Reference" "#PWR131"
+		(property "Reference" "#PWR130"
 			(at 223.52 134.62 0)
 			(effects
@@
 			(project "DualCore6502Whole"
 				(path "/93e0914e-b2e9-49c2-95f2-7cc419f4ea20/659d2ec5-e43d-4409-be3e-c470dc127456"
-					(reference "#PWR131")
+					(reference "#PWR130")
 					(unit 1)
 				)
@@
 		(dnp no)
 		(fields_autoplaced yes)
-		(property "Reference" "#PWR125"
+		(property "Reference" "#PWR124"
 			(at 93.98 64.77 0)
 			(effects
@@
 			(project "DualCore6502Whole"
 				(path "/93e0914e-b2e9-49c2-95f2-7cc419f4ea20/659d2ec5-e43d-4409-be3e-c470dc127456"
-					(reference "#PWR125")
+					(reference "#PWR124")
 					(unit 1)
 				)
