File: schematics/DualCore6502Whole/acia.kicad_sch (KiCad schematic)
At the start: 12 parts, among them J5 RS232, U20 W65C51N, U21 MAX232, Y2 1.8432MHz

Commit message: Basic PCB layout
Parts:
- U19: renamed from U20; footprint Package_DIP:DIP-28_W15.24mm -> Package_DIP:DIP-28_W15.24mm_Socket
- U20: renamed from U21; footprint Package_DIP:DIP-16_W7.62mm -> Package_DIP:DIP-16_W7.62mm_Socket
- Y2: footprint Crystal:Crystal_HC49-U_Horizontal -> Crystal:Crystal_HC49-U_Vertical
- renumbered C22 to C21, C23 to C22, C24 to C23, C25 to C24, C26 to C25, C27 to C26, D9 to D8
Connections:
- net TX: now reaches U19.10 (TxD), U20.11 (T1IN)
- net RX: now reaches U19.12 (RxD), U20.12 (R1OUT)
Changed lines of the file:
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@@
+	)
+	(junction
+		(at 144.78 90.17)
+		(diameter 0)
+		(color 0 0 0 0)
 	)
 	(junction
@@
 	)
 	(junction
+		(at 137.16 110.49)
+		(diameter 0)
+		(color 0 0 0 0)
+	)
+	(junction
 		(at 115.57 113.03)
 		(diameter 0)
@@
 	(wire
 		(pts
+			(xy 137.16 110.49) (xy 133.35 110.49)
+		)
+		(stroke
+			(width 0)
+			(type default)
+		)
+	)
+	(wire
+		(pts
 			(xy 113.03 80.01) (xy 119.38 80.01)
 		)
@@
 		(pts
 			(xy 214.63 100.33) (xy 259.08 100.33)
+		)
+		(stroke
+			(width 0)
+			(type default)
+		)
+	)
+	(wire
+		(pts
+			(xy 144.78 90.17) (xy 148.59 90.17)
 		)
 		(stroke
@@
 				)
 				(justify right)
+				(hide yes)
+			)
+		)
+	)
+	(global_label "RX"
+		(shape input)
+		(at 133.35 110.49 180)
+		(fields_autoplaced yes)
+		(effects
+			(font
+				(size 1.27 1.27)
+			)
+			(justify right)
+		)
+		(property "Intersheetrefs" "${INTERSHEET_REFS}"
+			(at 127.8853 110.49 0)
+			(effects
+				(font
+					(size 1.27 1.27)
+				)
+				(justify right)
+				(hide yes)
+			)
+		)
+	)
+	(global_label "TX"
+		(shape output)
+		(at 148.59 90.17 0)
+		(fields_autoplaced yes)
+		(effects
+			(font
+				(size 1.27 1.27)
+			)
+			(justify left)
+		)
+		(property "Intersheetrefs" "${INTERSHEET_REFS}"
+			(at 153.7523 90.17 0)
+			(effects
+				(font
+					(size 1.27 1.27)
+				)
+				(justify left)
 				(hide yes)
 			)
@@
 		(dnp no)
 		(fields_autoplaced yes)
-		(property "Reference" "U21"
+		(property "Reference" "U20"
 			(at 196.5041 67.31 0)
 			(effects
@@
 			)
 		)
-		(property "Footprint" "Package_DIP:DIP-16_W7.62mm"
+		(property "Footprint" "Package_DIP:DIP-16_W7.62mm_Socket"
 			(at 195.58 124.46 0)
 			(effects
@@
 			(project "DualCore6502Whole"
 				(path "/93e0914e-b2e9-49c2-95f2-7cc419f4ea20/659d2ec5-e43d-4409-be3e-c470dc127456"
-					(reference "U21")
+					(reference "U20")
 					(unit 1)
 				)
@@
 		(dnp no)
 		(fields_autoplaced yes)
-		(property "Reference" "U20"
+		(property "Reference" "U19"
 			(at 96.1741 60.96 0)
 			(effects
@@
 			)
 		)
-		(property "Footprint" "Package_DIP:DIP-28_W15.24mm"
+		(property "Footprint" "Package_DIP:DIP-28_W15.24mm_Socket"
 			(at 93.98 93.98 0)
 			(effects
@@
 			(project ""
 				(path "/93e0914e-b2e9-49c2-95f2-7cc419f4ea20/659d2ec5-e43d-4409-be3e-c470dc127456"
-					(reference "U20")
+					(reference "U19")
 					(unit 1)
 				)
@@
 		(dnp no)
 		(fields_autoplaced yes)
-		(property "Reference" "D9"
+		(property "Reference" "D8"
 			(at 54.9275 71.12 0)
 			(effects
@@
 			(project "DualCore6502Whole"
 				(path "/93e0914e-b2e9-49c2-95f2-7cc419f4ea20/659d2ec5-e43d-4409-be3e-c470dc127456"
-					(reference "D9")
+					(reference "D8")
 					(unit 1)
 				)
@@
 		(dnp no)
 		(fields_autoplaced yes)
-		(property "Reference" "C24"
+		(property "Reference" "C23"
 			(at 168.91 77.47 0)
 			(effects
@@
 			(project "DualCore6502Whole"
 				(path "/93e0914e-b2e9-49c2-95f2-7cc419f4ea20/659d2ec5-e43d-4409-be3e-c470dc127456"
-					(reference "C24")
+					(reference "C23")
 					(unit 1)
 				)
@@
 		(dnp no)
 		(fields_autoplaced yes)
-		(property "Reference" "C27"
+		(property "Reference" "C26"
 			(at 238.76 123.19 0)
 			(effects
@@
 			(project "DualCore6502Whole"
 				(path "/93e0914e-b2e9-49c2-95f2-7cc419f4ea20/659d2ec5-e43d-4409-be3e-c470dc127456"
-					(reference "C27")
+					(reference "C26")
 					(unit 1)
 				)
@@
 		(dnp no)
 		(fields_autoplaced yes)
-		(property "Reference" "#PWR126"
+		(property "Reference" "#PWR122"
 			(at 115.57 124.46 0)
 			(effects
@@
 			(project "DualCore6502Whole"
 				(path "/93e0914e-b2e9-49c2-95f2-7cc419f4ea20/659d2ec5-e43d-4409-be3e-c470dc127456"
-					(reference "#PWR126")
+					(reference "#PWR122")
 					(unit 1)
 				)
@@
 		(dnp no)
 		(fields_autoplaced yes)
-		(property "Reference" "#PWR123"
+		(property "Reference" "#PWR119"
 			(at 73.66 59.69 0)
 			(effects
@@
 			(project "DualCore6502Whole"
 				(path "/93e0914e-b2e9-49c2-95f2-7cc419f4ea20/659d2ec5-e43d-4409-be3e-c470dc127456"
-					(reference "#PWR123")
+					(reference "#PWR119")
 					(unit 1)
 				)
@@
 		(dnp no)
 		(fields_autoplaced yes)
-		(property "Reference" "#PWR127"
+		(property "Reference" "#PWR123"
 			(at 149.86 81.28 0)
 			(effects
@@
 			(project "DualCore6502Whole"
 				(path "/93e0914e-b2e9-49c2-95f2-7cc419f4ea20/659d2ec5-e43d-4409-be3e-c470dc127456"
-					(reference "#PWR127")
+					(reference "#PWR123")
 					(unit 1)
 				)
@@
 		(dnp no)
 		(fields_autoplaced yes)
-		(property "Reference" "C25"
+		(property "Reference" "C24"
 			(at 227.33 123.19 0)
 			(effects
@@
 			(project "DualCore6502Whole"
 				(path "/93e0914e-b2e9-49c2-95f2-7cc419f4ea20/659d2ec5-e43d-4409-be3e-c470dc127456"
-					(reference "C25")
+					(reference "C24")
 					(unit 1)
 				)
@@
 		(dnp no)
 		(fields_autoplaced yes)
-		(property "Reference" "#PWR122"
+		(property "Reference" "#PWR118"
 			(at 73.66 49.53 0)
 			(effects
@@
 			(project ""
 				(path "/93e0914e-b2e9-49c2-95f2-7cc419f4ea20/659d2ec5-e43d-4409-be3e-c470dc127456"
-					(reference "#PWR122")
+					(reference "#PWR118")
 					(unit 1)
 				)
@@
 		(dnp no)
 		(fields_autoplaced yes)
-		(property "Reference" "C22"
+		(property "Reference" "C21"
 			(at 77.47 48.26 0)
 			(effects
@@
 			(project "DualCore6502Whole"
 				(path "/93e0914e-b2e9-49c2-95f2-7cc419f4ea20/659d2ec5-e43d-4409-be3e-c470dc127456"
-					(reference "C22")
+					(reference "C21")
 					(unit 1)
 				)
@@
 		(dnp no)
 		(fields_autoplaced yes)
-		(property "Reference" "#PWR129"
+		(property "Reference" "#PWR125"
 			(at 194.31 134.62 0)
 			(effects
@@
 			(project "DualCore6502Whole"
 				(path "/93e0914e-b2e9-49c2-95f2-7cc419f4ea20/659d2ec5-e43d-4409-be3e-c470dc127456"
-					(reference "#PWR129")
+					(reference "#PWR125")
 					(unit 1)
 				)
@@
 		(dnp no)
 		(fields_autoplaced yes)
-		(property "Reference" "#PWR132"
+		(property "Reference" "#PWR128"
 			(at 256.54 124.46 0)
 			(effects
@@
 			(project "DualCore6502Whole"
 				(path "/93e0914e-b2e9-49c2-95f2-7cc419f4ea20/659d2ec5-e43d-4409-be3e-c470dc127456"
-					(reference "#PWR132")
+					(reference "#PWR128")
 					(unit 1)
 				)
@@
 		(fields_autoplaced yes)
 		(property "Reference" "Y2"
-			(at 134.62 69.85 90)
+			(at 134.62 69.8499 90)
 			(effects
 				(font
@@
 		)
 		(property "Value" "1.8432MHz"
-			(at 134.62 72.39 90)
+			(at 134.62 72.3899 90)
 			(effects
 				(font
@@
 			)
 		)
-		(property "Footprint" "Crystal:Crystal_HC49-U_Horizontal"
+		(property "Footprint" "Crystal:Crystal_HC49-U_Vertical"
 			(at 130.81 71.12 0)
 			(effects
@@
 		(dnp no)
 		(fields_autoplaced yes)
-		(property "Reference" "#PWR131"
+		(property "Reference" "#PWR127"
 			(at 234.95 134.62 0)
 			(effects
@@
 			(project "DualCore6502Whole"
 				(path "/93e0914e-b2e9-49c2-95f2-7cc419f4ea20/659d2ec5-e43d-4409-be3e-c470dc127456"
-					(reference "#PWR131")
+					(reference "#PWR127")
 					(unit 1)
 				)
@@
 		(dnp no)
 		(fields_autoplaced yes)
-		(property "Reference" "#PWR128"
+		(property "Reference" "#PWR124"
 			(at 194.31 71.12 0)
 			(effects
@@
 			(project "DualCore6502Whole"
 				(path "/93e0914e-b2e9-49c2-95f2-7cc419f4ea20/659d2ec5-e43d-4409-be3e-c470dc127456"
-					(reference "#PWR128")
+					(reference "#PWR124")
 					(unit 1)
 				)
@@
 		(dnp no)
 		(fields_autoplaced yes)
-		(property "Reference" "#PWR125"
+		(property "Reference" "#PWR121"
 			(at 93.98 140.97 0)
 			(effects
@@
 			(project ""
 				(path "/93e0914e-b2e9-49c2-95f2-7cc419f4ea20/659d2ec5-e43d-4409-be3e-c470dc127456"
-					(reference "#PWR125")
+					(reference "#PWR121")
 					(unit 1)
 				)
@@
 		(dnp no)
 		(fields_autoplaced yes)
-		(property "Reference" "C26"
+		(property "Reference" "C25"
 			(at 228.6 77.47 0)
 			(effects
@@
 			(project "DualCore6502Whole"
 				(path "/93e0914e-b2e9-49c2-95f2-7cc419f4ea20/659d2ec5-e43d-4409-be3e-c470dc127456"
-					(reference "C26")
+					(reference "C25")
 					(unit 1)
 				)
@@
 		(dnp no)
 		(fields_autoplaced yes)
-		(property "Reference" "#PWR130"
+		(property "Reference" "#PWR126"
 			(at 223.52 134.62 0)
 			(effects
@@
 			(project "DualCore6502Whole"
 				(path "/93e0914e-b2e9-49c2-95f2-7cc419f4ea20/659d2ec5-e43d-4409-be3e-c470dc127456"
-					(reference "#PWR130")
+					(reference "#PWR126")
 					(unit 1)
 				)
@@
 		(dnp no)
 		(fields_autoplaced yes)
-		(property "Reference" "#PWR124"
+		(property "Reference" "#PWR120"
 			(at 93.98 64.77 0)
 			(effects
@@
 			(project "DualCore6502Whole"
 				(path "/93e0914e-b2e9-49c2-95f2-7cc419f4ea20/659d2ec5-e43d-4409-be3e-c470dc127456"
-					(reference "#PWR124")
+					(reference "#PWR120")
 					(unit 1)
 				)
@@
 		(dnp no)
 		(fields_autoplaced yes)
-		(property "Reference" "C23"
+		(property "Reference" "C22"
 			(at 153.67 69.85 0)
 			(effects
@@
 			(project "DualCore6502Whole"
 				(path "/93e0914e-b2e9-49c2-95f2-7cc419f4ea20/659d2ec5-e43d-4409-be3e-c470dc127456"
-					(reference "C23")
+					(reference "C22")
 					(unit 1)
 				)
