File: schematics/DualCore6502Whole/address_decoding.kicad_sch (KiCad schematic)
At the start: 5 parts, among them U12 74HC00, U13 74HC138, U5 74HC08

Commit message: Remove the need to multiplex the control lines
Parts:
- renumbered C14 to C13, C15 to C14, U12 to U11, U13 to U12, U5 to U4
Changed lines of the file:
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@@
 		(dnp no)
 		(fields_autoplaced yes)
-		(property "Reference" "U5"
+		(property "Reference" "U4"
 			(at 124.4517 109.22 0)
 			(effects
@@
 			(project "DualCore6502Whole"
 				(path "/93e0914e-b2e9-49c2-95f2-7cc419f4ea20/c648dfd0-2e47-4168-b72a-602e847f0b30"
-					(reference "U5")
+					(reference "U4")
 					(unit 1)
 				)
@@
 		(dnp no)
 		(fields_autoplaced yes)
-		(property "Reference" "U12"
+		(property "Reference" "U11"
 			(at 48.26 158.7499 0)
 			(effects
@@
 			(project "DualCore6502Whole"
 				(path "/93e0914e-b2e9-49c2-95f2-7cc419f4ea20/c648dfd0-2e47-4168-b72a-602e847f0b30"
-					(reference "U12")
+					(reference "U11")
 					(unit 5)
 				)
@@
 		(dnp no)
 		(fields_autoplaced yes)
-		(property "Reference" "#PWR76"
+		(property "Reference" "#PWR69"
 			(at 81.28 123.19 0)
 			(effects
@@
 			(project "DualCore6502Whole"
 				(path "/93e0914e-b2e9-49c2-95f2-7cc419f4ea20/c648dfd0-2e47-4168-b72a-602e847f0b30"
-					(reference "#PWR76")
+					(reference "#PWR69")
 					(unit 1)
 				)
@@
 		(dnp no)
 		(fields_autoplaced yes)
-		(property "Reference" "U12"
+		(property "Reference" "U11"
 			(at 124.4517 67.31 0)
 			(effects
@@
 			(project "DualCore6502Whole"
 				(path "/93e0914e-b2e9-49c2-95f2-7cc419f4ea20/c648dfd0-2e47-4168-b72a-602e847f0b30"
-					(reference "U12")
+					(reference "U11")
 					(unit 3)
 				)
@@
 		(dnp no)
 		(fields_autoplaced yes)
-		(property "Reference" "#PWR72"
+		(property "Reference" "#PWR65"
 			(at 41.91 179.07 0)
 			(effects
@@
 			(project "DualCore6502Whole"
 				(path "/93e0914e-b2e9-49c2-95f2-7cc419f4ea20/c648dfd0-2e47-4168-b72a-602e847f0b30"
-					(reference "#PWR72")
+					(reference "#PWR65")
 					(unit 1)
 				)
@@
 		(dnp no)
 		(fields_autoplaced yes)
-		(property "Reference" "C14"
+		(property "Reference" "C13"
 			(at 66.04 158.75 0)
 			(effects
@@
 			(project "DualCore6502Whole"
 				(path "/93e0914e-b2e9-49c2-95f2-7cc419f4ea20/c648dfd0-2e47-4168-b72a-602e847f0b30"
-					(reference "C14")
+					(reference "C13")
 					(unit 1)
 				)
@@
 		(dnp no)
 		(fields_autoplaced yes)
-		(property "Reference" "#PWR74"
+		(property "Reference" "#PWR67"
 			(at 62.23 170.18 0)
 			(effects
@@
 			(project "DualCore6502Whole"
 				(path "/93e0914e-b2e9-49c2-95f2-7cc419f4ea20/c648dfd0-2e47-4168-b72a-602e847f0b30"
-					(reference "#PWR74")
+					(reference "#PWR67")
 					(unit 1)
 				)
@@
 		(dnp no)
 		(fields_autoplaced yes)
-		(property "Reference" "#PWR75"
+		(property "Reference" "#PWR68"
 			(at 81.28 81.28 0)
 			(effects
@@
 			(project "DualCore6502Whole"
 				(path "/93e0914e-b2e9-49c2-95f2-7cc419f4ea20/c648dfd0-2e47-4168-b72a-602e847f0b30"
-					(reference "#PWR75")
+					(reference "#PWR68")
 					(unit 1)
 				)
@@
 		(dnp no)
 		(fields_autoplaced yes)
-		(property "Reference" "U12"
+		(property "Reference" "U11"
 			(at 90.1617 90.17 0)
 			(effects
@@
 			(project "DualCore6502Whole"
 				(path "/93e0914e-b2e9-49c2-95f2-7cc419f4ea20/c648dfd0-2e47-4168-b72a-602e847f0b30"
-					(reference "U12")
+					(reference "U11")
 					(unit 1)
 				)
@@
 		(dnp no)
 		(fields_autoplaced yes)
-		(property "Reference" "#PWR80"
+		(property "Reference" "#PWR73"
 			(at 186.69 114.3 0)
 			(effects
@@
 			(project "DualCore6502Whole"
 				(path "/93e0914e-b2e9-49c2-95f2-7cc419f4ea20/c648dfd0-2e47-4168-b72a-602e847f0b30"
-					(reference "#PWR80")
+					(reference "#PWR73")
 					(unit 1)
 				)
@@
 		(dnp no)
 		(fields_autoplaced yes)
-		(property "Reference" "U12"
+		(property "Reference" "U11"
 			(at 90.1617 69.85 0)
 			(effects
@@
 			(project "DualCore6502Whole"
 				(path "/93e0914e-b2e9-49c2-95f2-7cc419f4ea20/c648dfd0-2e47-4168-b72a-602e847f0b30"
-					(reference "U12")
+					(reference "U11")
 					(unit 4)
 				)
@@
 		(dnp no)
 		(fields_autoplaced yes)
-		(property "Reference" "#PWR71"
+		(property "Reference" "#PWR64"
 			(at 41.91 151.13 0)
 			(effects
@@
 			(project "DualCore6502Whole"
 				(path "/93e0914e-b2e9-49c2-95f2-7cc419f4ea20/c648dfd0-2e47-4168-b72a-602e847f0b30"
-					(reference "#PWR71")
+					(reference "#PWR64")
 					(unit 1)
 				)
@@
 		(dnp no)
 		(fields_autoplaced yes)
-		(property "Reference" "#PWR79"
+		(property "Reference" "#PWR72"
 			(at 186.69 78.74 0)
 			(effects
@@
 			(project "DualCore6502Whole"
 				(path "/93e0914e-b2e9-49c2-95f2-7cc419f4ea20/c648dfd0-2e47-4168-b72a-602e847f0b30"
-					(reference "#PWR79")
+					(reference "#PWR72")
 					(unit 1)
 				)
@@
 		(dnp no)
 		(fields_autoplaced yes)
-		(property "Reference" "#PWR78"
+		(property "Reference" "#PWR71"
 			(at 186.69 63.5 0)
 			(effects
@@
 			(project "DualCore6502Whole"
 				(path "/93e0914e-b2e9-49c2-95f2-7cc419f4ea20/c648dfd0-2e47-4168-b72a-602e847f0b30"
-					(reference "#PWR78")
+					(reference "#PWR71")
 					(unit 1)
 				)
@@
 		(dnp no)
 		(fields_autoplaced yes)
-		(property "Reference" "U12"
+		(property "Reference" "U11"
 			(at 90.1617 111.76 0)
 			(effects
@@
 			(project "DualCore6502Whole"
 				(path "/93e0914e-b2e9-49c2-95f2-7cc419f4ea20/c648dfd0-2e47-4168-b72a-602e847f0b30"
-					(reference "U12")
+					(reference "U11")
 					(unit 2)
 				)
@@
 		(dnp no)
 		(fields_autoplaced yes)
-		(property "Reference" "#PWR77"
+		(property "Reference" "#PWR70"
 			(at 186.69 53.34 0)
 			(effects
@@
 			(project "DualCore6502Whole"
 				(path "/93e0914e-b2e9-49c2-95f2-7cc419f4ea20/c648dfd0-2e47-4168-b72a-602e847f0b30"
-					(reference "#PWR77")
+					(reference "#PWR70")
 					(unit 1)
 				)
@@
 		(dnp no)
 		(fields_autoplaced yes)
-		(property "Reference" "U13"
+		(property "Reference" "U12"
 			(at 188.8841 74.93 0)
 			(effects
@@
 			(project ""
 				(path "/93e0914e-b2e9-49c2-95f2-7cc419f4ea20/c648dfd0-2e47-4168-b72a-602e847f0b30"
-					(reference "U13")
+					(reference "U12")
 					(unit 1)
 				)
@@
 		(dnp no)
 		(fields_autoplaced yes)
-		(property "Reference" "C15"
+		(property "Reference" "C14"
 			(at 190.5 52.07 0)
 			(effects
@@
 			(project "DualCore6502Whole"
 				(path "/93e0914e-b2e9-49c2-95f2-7cc419f4ea20/c648dfd0-2e47-4168-b72a-602e847f0b30"
-					(reference "C15")
+					(reference "C14")
 					(unit 1)
 				)
@@
 		(dnp no)
 		(fields_autoplaced yes)
-		(property "Reference" "#PWR73"
+		(property "Reference" "#PWR66"
 			(at 62.23 160.02 0)
 			(effects
@@
 			(project "DualCore6502Whole"
 				(path "/93e0914e-b2e9-49c2-95f2-7cc419f4ea20/c648dfd0-2e47-4168-b72a-602e847f0b30"
-					(reference "#PWR73")
-					(unit 1)
-				)
+					(reference "#PWR66")
+					(unit 1)
+				)

Commit message: Add simpler I/O outputs as an alternative to the VIA
Parts:
- removed U4: 74HC08, Package_DIP:DIP-14_W7.62mm, symbol 74xx:74LS08
- added C14: 100nF, Capacitor_THT:C_Disc_D5.0mm_W2.5mm_P5.00mm, symbol Device:C
- added U12: 74HC00, Package_DIP:DIP-14_W7.62mm, symbol 74xx:74LS00
- renumbered C14 to C15, U12 to U13
Connections:
- net +5V: now also C14.1, U12.14 (VCC), U12.9
- net A15: now also U12.12
- net GND: now also C14.2, U12.7 (GND)
- net IO_CS: now also U12.8
- net at U11.6: now also U12.13
- new net: U12.10, U12.11

Commit message: Update the schematic
Parts:
- removed C14: 100nF, Capacitor_THT:C_Disc_D5.0mm_W2.5mm_P5.00mm, symbol Device:C
- removed U12: 74HC00, Package_DIP:DIP-14_W7.62mm, symbol 74xx:74LS00
- added U8: 74HC86, Package_DIP:DIP-14_W7.62mm, symbol 74xx:74LS86
- renumbered C15 to C14, U13 to U12
Connections:
- net +5V: now also U8.2, U8.4; no longer U11.5
- net A14: now also U8.1; no longer U11.4
- net A15: now also U11.4
- net IO_CS: now also U8.6
- net at U11.6: now also U8.5
- new net: U11.5, U8.3
Other:
- note added: "Memory Map: $0000 - $01FF - Zero page and stack for CPU1 $0200 - $03FF - Zero page and stack for CPU2 $0400 - $7FFF - Shared RAM $8000 - $8FFF - I/O Devices $9000 - $BFFF - Spare $C000 - $FFFF - This CPU's ROM"
- note removed: "Memory Map: $0000 - $3FFF - This CPU's RAM $4000 - $7FFF - Other CPU's RAM $8000 - $8FFF - I/O Devices $9000 - $BFFF - Spare $C000 - $FFFF - This CPU's ROM"
- title: (none) -> Dual Core 65C02 Computer
- moved on the sheet: U11B

Commit message: Update schematic and add 1ms NMI tick
Connections:
- net A12: now also U12.4 (E1); no longer U12.5 (E2)
- net A13: now also U12.5 (E2); no longer U12.4 (E1)
Changed lines of the file:
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@@
 	)
 	(label "A12"
-		(at 166.37 97.79 0)
+		(at 166.37 100.33 0)
 		(effects
 			(font
@@
 	)
 	(label "A13"
-		(at 166.37 100.33 0)
+		(at 166.37 97.79 0)
 		(effects
 			(font
@@
 		(dnp no)
 		(fields_autoplaced yes)
-		(property "Reference" "#PWR73"
+		(property "Reference" "#PWR72"
 			(at 81.28 123.19 0)
 			(effects
@@
 			(project "DualCore6502Whole"
 				(path "/93e0914e-b2e9-49c2-95f2-7cc419f4ea20/c648dfd0-2e47-4168-b72a-602e847f0b30"
-					(reference "#PWR73")
+					(reference "#PWR72")
 					(unit 1)
 				)
@@
 		(dnp no)
 		(fields_autoplaced yes)
-		(property "Reference" "#PWR69"
+		(property "Reference" "#PWR68"
 			(at 41.91 179.07 0)
 			(effects
@@
 			(project "DualCore6502Whole"
 				(path "/93e0914e-b2e9-49c2-95f2-7cc419f4ea20/c648dfd0-2e47-4168-b72a-602e847f0b30"
-					(reference "#PWR69")
+					(reference "#PWR68")
 					(unit 1)
 				)
@@
 		(dnp no)
 		(fields_autoplaced yes)
-		(property "Reference" "#PWR71"
+		(property "Reference" "#PWR70"
 			(at 62.23 170.18 0)
 			(effects
@@
 			(project "DualCore6502Whole"
 				(path "/93e0914e-b2e9-49c2-95f2-7cc419f4ea20/c648dfd0-2e47-4168-b72a-602e847f0b30"
-					(reference "#PWR71")
+					(reference "#PWR70")
 					(unit 1)
 				)
@@
 		(dnp no)
 		(fields_autoplaced yes)
-		(property "Reference" "#PWR72"
+		(property "Reference" "#PWR71"
 			(at 81.28 81.28 0)
 			(effects
@@
 			(project "DualCore6502Whole"
 				(path "/93e0914e-b2e9-49c2-95f2-7cc419f4ea20/c648dfd0-2e47-4168-b72a-602e847f0b30"
-					(reference "#PWR72")
+					(reference "#PWR71")
 					(unit 1)
 				)
@@
 		(dnp no)
 		(fields_autoplaced yes)
-		(property "Reference" "#PWR78"
+		(property "Reference" "#PWR77"
 			(at 186.69 114.3 0)
 			(effects
@@
 			(project "DualCore6502Whole"
 				(path "/93e0914e-b2e9-49c2-95f2-7cc419f4ea20/c648dfd0-2e47-4168-b72a-602e847f0b30"
-					(reference "#PWR78")
+					(reference "#PWR77")
 					(unit 1)
 				)
@@
 		(dnp no)
 		(fields_autoplaced yes)
-		(property "Reference" "#PWR68"
+		(property "Reference" "#PWR67"
 			(at 41.91 151.13 0)
 			(effects
@@
 			(project "DualCore6502Whole"
 				(path "/93e0914e-b2e9-49c2-95f2-7cc419f4ea20/c648dfd0-2e47-4168-b72a-602e847f0b30"
-					(reference "#PWR68")
+					(reference "#PWR67")
 					(unit 1)
 				)
@@
 		(dnp no)
 		(fields_autoplaced yes)
-		(property "Reference" "#PWR77"
+		(property "Reference" "#PWR76"
 			(at 186.69 78.74 0)
 			(effects
@@
 			(project "DualCore6502Whole"
 				(path "/93e0914e-b2e9-49c2-95f2-7cc419f4ea20/c648dfd0-2e47-4168-b72a-602e847f0b30"
-					(reference "#PWR77")
+					(reference "#PWR76")
 					(unit 1)
 				)
@@
 		(dnp no)
 		(fields_autoplaced yes)
-		(property "Reference" "#PWR74"
+		(property "Reference" "#PWR73"
 			(at 143.51 113.03 0)
 			(effects
@@
 			(project "DualCore6502Whole"
 				(path "/93e0914e-b2e9-49c2-95f2-7cc419f4ea20/c648dfd0-2e47-4168-b72a-602e847f0b30"
-					(reference "#PWR74")
+					(reference "#PWR73")
 					(unit 1)
 				)
@@
 		(dnp no)
 		(fields_autoplaced yes)
-		(property "Reference" "#PWR76"
+		(property "Reference" "#PWR75"
 			(at 186.69 63.5 0)
 			(effects
@@
 			(project "DualCore6502Whole"
 				(path "/93e0914e-b2e9-49c2-95f2-7cc419f4ea20/c648dfd0-2e47-4168-b72a-602e847f0b30"
-					(reference "#PWR76")
+					(reference "#PWR75")
 					(unit 1)
 				)
@@
 		(dnp no)
 		(fields_autoplaced yes)
-		(property "Reference" "#PWR75"
+		(property "Reference" "#PWR74"
 			(at 186.69 53.34 0)
 			(effects
@@
 			(project "DualCore6502Whole"
 				(path "/93e0914e-b2e9-49c2-95f2-7cc419f4ea20/c648dfd0-2e47-4168-b72a-602e847f0b30"
-					(reference "#PWR75")
+					(reference "#PWR74")
 					(unit 1)
 				)
@@
 		(dnp no)
 		(fields_autoplaced yes)
-		(property "Reference" "#PWR70"
+		(property "Reference" "#PWR69"
 			(at 62.23 160.02 0)
 			(effects
@@
 			(project "DualCore6502Whole"
 				(path "/93e0914e-b2e9-49c2-95f2-7cc419f4ea20/c648dfd0-2e47-4168-b72a-602e847f0b30"
-					(reference "#PWR70")
+					(reference "#PWR69")
 					(unit 1)
 				)

Commit message: Basic PCB layout
Parts:
- U10: renamed from U11; footprint Package_DIP:DIP-14_W7.62mm -> Package_DIP:DIP-14_W7.62mm_Socket
- U11: renamed from U12; footprint Package_DIP:DIP-16_W7.62mm -> Package_DIP:DIP-16_W7.62mm_Socket
- U7: renamed from U8; footprint Package_DIP:DIP-14_W7.62mm -> Package_DIP:DIP-14_W7.62mm_Socket
- renumbered C13 to C12, C14 to C13
Changed lines of the file:
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@@
 		(dnp no)
 		(fields_autoplaced yes)
-		(property "Reference" "U11"
+		(property "Reference" "U10"
 			(at 48.26 158.7499 0)
 			(effects
@@
 			)
 		)
-		(property "Footprint" "Package_DIP:DIP-14_W7.62mm"
+		(property "Footprint" "Package_DIP:DIP-14_W7.62mm_Socket"
 			(at 41.91 160.02 0)
 			(effects
@@
 			(project "DualCore6502Whole"
 				(path "/93e0914e-b2e9-49c2-95f2-7cc419f4ea20/c648dfd0-2e47-4168-b72a-602e847f0b30"
-					(reference "U11")
+					(reference "U10")
 					(unit 5)
 				)
@@
 		(dnp no)
 		(fields_autoplaced yes)
-		(property "Reference" "#PWR72"
+		(property "Reference" "#PWR68"
 			(at 81.28 123.19 0)
 			(effects
@@
 			(project "DualCore6502Whole"
 				(path "/93e0914e-b2e9-49c2-95f2-7cc419f4ea20/c648dfd0-2e47-4168-b72a-602e847f0b30"
-					(reference "#PWR72")
+					(reference "#PWR68")
 					(unit 1)
 				)
@@
 		(dnp no)
 		(fields_autoplaced yes)
-		(property "Reference" "U11"
+		(property "Reference" "U10"
 			(at 124.4517 67.31 0)
 			(effects
@@
 			)
 		)
-		(property "Footprint" "Package_DIP:DIP-14_W7.62mm"
+		(property "Footprint" "Package_DIP:DIP-14_W7.62mm_Socket"
 			(at 124.46 76.2 0)
 			(effects
@@
 			(project "DualCore6502Whole"
 				(path "/93e0914e-b2e9-49c2-95f2-7cc419f4ea20/c648dfd0-2e47-4168-b72a-602e847f0b30"
-					(reference "U11")
+					(reference "U10")
 					(unit 3)
 				)
@@
 		(dnp no)
 		(fields_autoplaced yes)
-		(property "Reference" "#PWR68"
+		(property "Reference" "#PWR64"
 			(at 41.91 179.07 0)
 			(effects
@@
 			(project "DualCore6502Whole"
 				(path "/93e0914e-b2e9-49c2-95f2-7cc419f4ea20/c648dfd0-2e47-4168-b72a-602e847f0b30"
-					(reference "#PWR68")
+					(reference "#PWR64")
 					(unit 1)
 				)
@@
 		(dnp no)
 		(fields_autoplaced yes)
-		(property "Reference" "C13"
+		(property "Reference" "C12"
 			(at 66.04 158.75 0)
 			(effects
@@
 			(project "DualCore6502Whole"
 				(path "/93e0914e-b2e9-49c2-95f2-7cc419f4ea20/c648dfd0-2e47-4168-b72a-602e847f0b30"
-					(reference "C13")
+					(reference "C12")
 					(unit 1)
 				)
@@
 		(dnp no)
 		(fields_autoplaced yes)
-		(property "Reference" "U8"
+		(property "Reference" "U7"
 			(at 89.8652 111.76 0)
 			(effects
@@
 			)
 		)
-		(property "Footprint" "Package_DIP:DIP-14_W7.62mm"
+		(property "Footprint" "Package_DIP:DIP-14_W7.62mm_Socket"
 			(at 90.17 120.65 0)
 			(effects
@@
 			(project "DualCore6502Whole"
 				(path "/93e0914e-b2e9-49c2-95f2-7cc419f4ea20/c648dfd0-2e47-4168-b72a-602e847f0b30"
-					(reference "U8")
+					(reference "U7")
 					(unit 1)
 				)
@@
 		(dnp no)
 		(fields_autoplaced yes)
-		(property "Reference" "#PWR70"
+		(property "Reference" "#PWR66"
 			(at 62.23 170.18 0)
 			(effects
@@
 			(project "DualCore6502Whole"
 				(path "/93e0914e-b2e9-49c2-95f2-7cc419f4ea20/c648dfd0-2e47-4168-b72a-602e847f0b30"
-					(reference "#PWR70")
+					(reference "#PWR66")
 					(unit 1)
 				)
@@
 		(dnp no)
 		(fields_autoplaced yes)
-		(property "Reference" "U8"
+		(property "Reference" "U7"
 			(at 148.2852 106.68 0)
 			(effects
@@
 			)
 		)
-		(property "Footprint" "Package_DIP:DIP-14_W7.62mm"
+		(property "Footprint" "Package_DIP:DIP-14_W7.62mm_Socket"
 			(at 148.59 115.57 0)
 			(effects
@@
 			(project "DualCore6502Whole"
 				(path "/93e0914e-b2e9-49c2-95f2-7cc419f4ea20/c648dfd0-2e47-4168-b72a-602e847f0b30"
-					(reference "U8")
+					(reference "U7")
 					(unit 2)
 				)
@@
 		(dnp no)
 		(fields_autoplaced yes)
-		(property "Reference" "#PWR71"
+		(property "Reference" "#PWR67"
 			(at 81.28 81.28 0)
 			(effects
@@
 			(project "DualCore6502Whole"
 				(path "/93e0914e-b2e9-49c2-95f2-7cc419f4ea20/c648dfd0-2e47-4168-b72a-602e847f0b30"
-					(reference "#PWR71")
+					(reference "#PWR67")
 					(unit 1)
 				)
@@
 		(dnp no)
 		(fields_autoplaced yes)
-		(property "Reference" "U11"
+		(property "Reference" "U10"
 			(at 90.1617 90.17 0)
 			(effects
@@
 			)
 		)
-		(property "Footprint" "Package_DIP:DIP-14_W7.62mm"
+		(property "Footprint" "Package_DIP:DIP-14_W7.62mm_Socket"
 			(at 90.17 99.06 0)
 			(effects
@@
 			(project "DualCore6502Whole"
 				(path "/93e0914e-b2e9-49c2-95f2-7cc419f4ea20/c648dfd0-2e47-4168-b72a-602e847f0b30"
-					(reference "U11")
+					(reference "U10")
 					(unit 1)
 				)
@@
 		(dnp no)
 		(fields_autoplaced yes)
-		(property "Reference" "#PWR77"
+		(property "Reference" "#PWR73"
 			(at 186.69 114.3 0)
 			(effects
@@
 			(project "DualCore6502Whole"
 				(path "/93e0914e-b2e9-49c2-95f2-7cc419f4ea20/c648dfd0-2e47-4168-b72a-602e847f0b30"
-					(reference "#PWR77")
+					(reference "#PWR73")
 					(unit 1)
 				)
@@
 		(dnp no)
 		(fields_autoplaced yes)
-		(property "Reference" "U11"
+		(property "Reference" "U10"
 			(at 90.1617 69.85 0)
 			(effects
@@
 			)
 		)
-		(property "Footprint" "Package_DIP:DIP-14_W7.62mm"
+		(property "Footprint" "Package_DIP:DIP-14_W7.62mm_Socket"
 			(at 90.17 78.74 0)
 			(effects
@@
 			(project "DualCore6502Whole"
 				(path "/93e0914e-b2e9-49c2-95f2-7cc419f4ea20/c648dfd0-2e47-4168-b72a-602e847f0b30"
-					(reference "U11")
+					(reference "U10")
 					(unit 4)
 				)
@@
 		(dnp no)
 		(fields_autoplaced yes)
-		(property "Reference" "#PWR67"
+		(property "Reference" "#PWR63"
 			(at 41.91 151.13 0)
 			(effects
@@
 			(project "DualCore6502Whole"
 				(path "/93e0914e-b2e9-49c2-95f2-7cc419f4ea20/c648dfd0-2e47-4168-b72a-602e847f0b30"
-					(reference "#PWR67")
+					(reference "#PWR63")
 					(unit 1)
 				)
@@
 		(dnp no)
 		(fields_autoplaced yes)
-		(property "Reference" "#PWR76"
+		(property "Reference" "#PWR72"
 			(at 186.69 78.74 0)
 			(effects
@@
 			(project "DualCore6502Whole"
 				(path "/93e0914e-b2e9-49c2-95f2-7cc419f4ea20/c648dfd0-2e47-4168-b72a-602e847f0b30"
-					(reference "#PWR76")
+					(reference "#PWR72")
 					(unit 1)
 				)
@@
 		(dnp no)
 		(fields_autoplaced yes)
-		(property "Reference" "#PWR73"
+		(property "Reference" "#PWR69"
 			(at 143.51 113.03 0)
 			(effects
@@
 			(project "DualCore6502Whole"
 				(path "/93e0914e-b2e9-49c2-95f2-7cc419f4ea20/c648dfd0-2e47-4168-b72a-602e847f0b30"
-					(reference "#PWR73")
+					(reference "#PWR69")
 					(unit 1)
 				)
@@
 		(dnp no)
 		(fields_autoplaced yes)
-		(property "Reference" "#PWR75"
+		(property "Reference" "#PWR71"
 			(at 186.69 63.5 0)
 			(effects
@@
 			(project "DualCore6502Whole"
 				(path "/93e0914e-b2e9-49c2-95f2-7cc419f4ea20/c648dfd0-2e47-4168-b72a-602e847f0b30"
-					(reference "#PWR75")
+					(reference "#PWR71")
 					(unit 1)
 				)
@@
 		(dnp no)
 		(fields_autoplaced yes)
-		(property "Reference" "U11"
+		(property "Reference" "U10"
 			(at 124.4517 109.22 0)
 			(effects
@@
 			)
 		)
-		(property "Footprint" "Package_DIP:DIP-14_W7.62mm"
+		(property "Footprint" "Package_DIP:DIP-14_W7.62mm_Socket"
 			(at 124.46 118.11 0)
 			(effects
@@
 			(project "DualCore6502Whole"
 				(path "/93e0914e-b2e9-49c2-95f2-7cc419f4ea20/c648dfd0-2e47-4168-b72a-602e847f0b30"
-					(reference "U11")
+					(reference "U10")
 					(unit 2)
 				)
@@
 		(dnp no)
 		(fields_autoplaced yes)
-		(property "Reference" "#PWR74"
+		(property "Reference" "#PWR70"
 			(at 186.69 53.34 0)
 			(effects
@@
 			(project "DualCore6502Whole"
 				(path "/93e0914e-b2e9-49c2-95f2-7cc419f4ea20/c648dfd0-2e47-4168-b72a-602e847f0b30"
-					(reference "#PWR74")
+					(reference "#PWR70")
 					(unit 1)
 				)
@@
 		(dnp no)
 		(fields_autoplaced yes)
-		(property "Reference" "U12"
+		(property "Reference" "U11"
 			(at 188.8841 74.93 0)
 			(effects
@@
 			)
 		)
-		(property "Footprint" "Package_DIP:DIP-16_W7.62mm"
+		(property "Footprint" "Package_DIP:DIP-16_W7.62mm_Socket"
 			(at 186.69 90.17 0)
 			(effects
@@
 			(project ""
 				(path "/93e0914e-b2e9-49c2-95f2-7cc419f4ea20/c648dfd0-2e47-4168-b72a-602e847f0b30"
-					(reference "U12")
+					(reference "U11")
 					(unit 1)
 				)
@@
 		(dnp no)
 		(fields_autoplaced yes)
-		(property "Reference" "C14"
+		(property "Reference" "C13"
 			(at 190.5 52.07 0)
 			(effects
@@
 			(project "DualCore6502Whole"
 				(path "/93e0914e-b2e9-49c2-95f2-7cc419f4ea20/c648dfd0-2e47-4168-b72a-602e847f0b30"
-					(reference "C14")
+					(reference "C13")
 					(unit 1)
 				)
@@
 		(dnp no)
 		(fields_autoplaced yes)
-		(property "Reference" "#PWR69"
+		(property "Reference" "#PWR65"
 			(at 62.23 160.02 0)
 			(effects
@@
 			(project "DualCore6502Whole"
 				(path "/93e0914e-b2e9-49c2-95f2-7cc419f4ea20/c648dfd0-2e47-4168-b72a-602e847f0b30"
-					(reference "#PWR69")
+					(reference "#PWR65")
 					(unit 1)
 				)
