File: schematics/DualCore6502Whole/clock.kicad_sch (KiCad schematic)
At the start: 9 parts, among them U5 74HC08, U6 74HC02, U7 74HC32, U8 74HC4017, Y1 12MHz

Commit message: Remove the need to multiplex the control lines
Parts:
- renumbered C7 to C6, C8 to C7, C9 to C8, C10 to C9, U5 to U4, U6 to U5, U7 to U6, U8 to U7
Connections:
- net CPU1_CLK: now also U6.13; no longer U6.12
- net CPU2_CLK: now also U6.12; no longer U6.13

Commit message: Add simpler I/O outputs as an alternative to the VIA
Parts:
- added unit 1 of U4
Connections:
- net GND: now also U4.1, U4.2
- no-connect marks 8 -> 9
Changed lines of the file:
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@@
 	(paper "A4")
+	(junction
+		(at 27.94 133.35)
+		(diameter 0)
+		(color 0 0 0 0)
+	)
+	(junction
+		(at 27.94 120.65)
+		(diameter 0)
+		(color 0 0 0 0)
+	)
 	(junction
 		(at 27.94 138.43)
@@
 		(at 123.19 46.99)
 	)
+	(no_connect
+		(at 46.99 118.11)
+	)
 	(polyline
 		(pts
@@
 		)
 	)
+	(wire
+		(pts
+			(xy 27.94 120.65) (xy 31.75 120.65)
+		)
+		(stroke
+			(width 0)
+			(type default)
+		)
+	)
 	(polyline
 		(pts
@@
 		)
 	)
+	(wire
+		(pts
+			(xy 27.94 120.65) (xy 27.94 133.35)
+		)
+		(stroke
+			(width 0)
+			(type default)
+		)
+	)
 	(polyline
 		(pts
@@
 		)
 	)
+	(wire
+		(pts
+			(xy 31.75 115.57) (xy 27.94 115.57)
+		)
+		(stroke
+			(width 0)
+			(type default)
+		)
+	)
 	(polyline
 		(pts
@@
 		(pts
 			(xy 96.52 104.648) (xy 96.52 108.458)
+		)
+		(stroke
+			(width 0)
+			(type default)
+		)
+	)
+	(wire
+		(pts
+			(xy 27.94 115.57) (xy 27.94 120.65)
 		)
 		(stroke
@@
 					(unit 1)
 				)
+			)
+		)
+	)
+	(symbol
+		(lib_id "74xx:74LS08")
+		(at 39.37 118.11 0)
+		(unit 1)
+		(exclude_from_sim no)
+		(in_bom yes)
+		(on_board yes)
+		(dnp no)
+		(fields_autoplaced yes)
+		(property "Reference" "U4"
+			(at 39.3617 109.22 0)
+			(effects
+				(font
+					(size 1.27 1.27)
+				)
+			)
+		)
+		(property "Value" "74HC08"
+			(at 39.3617 111.76 0)
+			(effects
+				(font
+					(size 1.27 1.27)
+				)
+			)
+		)
+		(property "Footprint" "Package_DIP:DIP-14_W7.62mm"
+			(at 39.37 118.11 0)
+			(effects
+				(font
+					(size 1.27 1.27)
+				)
+				(hide yes)
+			)
+		)
+		(property "Datasheet" "http://www.ti.com/lit/gpn/sn74LS08"
+			(at 39.37 118.11 0)
+			(effects
+				(font
+					(size 1.27 1.27)
+				)
+				(hide yes)
+			)
+		)
+		(property "Description" "Quad And2"
+			(at 39.37 118.11 0)
+			(effects
+				(font
+					(size 1.27 1.27)
+				)
+				(hide yes)
+			)
+		)
+		(pin "10"
+		)
+		(pin "3"
+		)
+		(pin "7"
+		)
+		(pin "8"
+		)
+		(pin "13"
+		)
+		(pin "6"
+		)
+		(pin "11"
+		)
+		(pin "9"
+		)
+		(pin "2"
+		)
+		(pin "5"
+		)
+		(pin "1"
+		)
+		(pin "4"
+		)
+		(pin "14"
+		)
+		(pin "12"
+		)
+		(instances
+			(project "DualCore6502Whole"
+				(path "/93e0914e-b2e9-49c2-95f2-7cc419f4ea20/a0d3e152-f132-475a-a70b-222ddccb1f8a"
+					(reference "U4")
+					(unit 1)
+				)

Commit message: Update the schematic
Parts:
- removed C8: 100nF, Capacitor_THT:C_Disc_D5.0mm_W2.5mm_P5.00mm, symbol Device:C
- removed U4: 74HC08, Package_DIP:DIP-14_W7.62mm, symbol 74xx:74LS08
- added unit 3 of U4
- added unit 4 of U4
- added unit 3 of U5
- added unit 1 of U5
- added unit 2 of U5
- renumbered C9 to C8, U5 to U4, U6 to U5, U7 to U6
Connections:
- net +5V: now also U4.11, U4.12, U4.8, U4.9
- net BUSEN_RESET: now also U4.2
- net BUSEN_SET: now also U4.6
- net CPU1_CLK: now also U5.3; no longer U5.13, U6.2 (Q1)
- net CPU2_CLK: now also U5.8; no longer U5.12, U6.10 (Q4)
- net GND: now also U5.2, U5.4, U5.5, U5.9
- net MAIN_CLK: now reaches U6.14 (CLK), Y1.8 (OUT)
- new net CPU1_CLK_RAW: U5.1, U5.13, U6.2 (Q1)
- new net CPU2_CLK_RAW: U5.10, U5.12, U6.10 (Q4)
- no-connect marks 9 -> 10
Other:
- note added: "Raw CPU1_CLK and CPU2_CLK are delayed by one gate delay to match timing with COMMON_CLK."
- title: (none) -> Dual Core 65C02 Computer
- moved on the sheet: U4A, U4B, U5D

Commit message: Update schematic and add 1ms NMI tick
Parts:
- removed unit 3 of U4
- removed unit 4 of U4
- renumbered U5 to U4, U4 to U5
Connections:
- no-connect marks 10 -> 8

Commit message: Basic PCB layout
Parts:
- U3: renamed from U4; footprint Package_DIP:DIP-14_W7.62mm -> Package_DIP:DIP-14_W7.62mm_Socket
- U4: renamed from U5; footprint Package_DIP:DIP-14_W7.62mm -> Package_DIP:DIP-14_W7.62mm_Socket
- U5: renamed from U6; footprint Package_DIP:DIP-16_W7.62mm -> Package_DIP:DIP-16_W7.62mm_Socket
- renumbered C6 to C5, C7 to C6, C8 to C7
