File: schematics/DualCore6502Whole/cpu2.kicad_sch (KiCad schematic)
At the start: 5 parts, among them U4 W65C02S

Commit message: Remove the need to multiplex the control lines
Parts:
- renumbered C6 to C5, U4 to U3
Connections:
- net CPU2_R/~{W} renamed R/~{W}
Changed lines of the file:
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@@
 		)
 	)
-	(global_label "CPU2_R{slash}~{W}"
+	(global_label "R{slash}~{W}"
 		(shape output)
 		(at 129.54 97.79 180)
@@
 		)
 		(property "Intersheetrefs" "${INTERSHEET_REFS}"
-			(at 116.4553 97.79 0)
+			(at 122.5029 97.79 0)
 			(effects
 				(font
@@
 		(dnp no)
 		(fields_autoplaced yes)
-		(property "Reference" "#PWR30"
+		(property "Reference" "#PWR23"
 			(at 120.65 46.99 0)
 			(effects
@@
 			(project "DualCore6502Whole"
 				(path "/93e0914e-b2e9-49c2-95f2-7cc419f4ea20/578e6b65-8887-41c5-b062-8f45f343257b"
-					(reference "#PWR30")
+					(reference "#PWR23")
 					(unit 1)
 				)
@@
 		(dnp no)
 		(fields_autoplaced yes)
-		(property "Reference" "#PWR32"
+		(property "Reference" "#PWR25"
 			(at 133.35 128.27 0)
 			(effects
@@
 			(project "DualCore6502Whole"
 				(path "/93e0914e-b2e9-49c2-95f2-7cc419f4ea20/578e6b65-8887-41c5-b062-8f45f343257b"
-					(reference "#PWR32")
+					(reference "#PWR25")
 					(unit 1)
 				)
@@
 		(dnp no)
 		(fields_autoplaced yes)
-		(property "Reference" "#PWR28"
+		(property "Reference" "#PWR21"
 			(at 88.9 81.28 0)
 			(effects
@@
 			(project "DualCore6502Whole"
 				(path "/93e0914e-b2e9-49c2-95f2-7cc419f4ea20/578e6b65-8887-41c5-b062-8f45f343257b"
-					(reference "#PWR28")
+					(reference "#PWR21")
 					(unit 1)
 				)
@@
 		(dnp no)
 		(fields_autoplaced yes)
-		(property "Reference" "#PWR31"
+		(property "Reference" "#PWR24"
 			(at 120.65 57.15 0)
 			(effects
@@
 			(project "DualCore6502Whole"
 				(path "/93e0914e-b2e9-49c2-95f2-7cc419f4ea20/578e6b65-8887-41c5-b062-8f45f343257b"
-					(reference "#PWR31")
+					(reference "#PWR24")
 					(unit 1)
 				)
@@
 		(dnp no)
 		(fields_autoplaced yes)
-		(property "Reference" "#PWR33"
+		(property "Reference" "#PWR26"
 			(at 149.86 62.23 0)
 			(effects
@@
 			(project "DualCore6502Whole"
 				(path "/93e0914e-b2e9-49c2-95f2-7cc419f4ea20/578e6b65-8887-41c5-b062-8f45f343257b"
-					(reference "#PWR33")
+					(reference "#PWR26")
 					(unit 1)
 				)
@@
 		(dnp no)
 		(fields_autoplaced yes)
-		(property "Reference" "#PWR29"
+		(property "Reference" "#PWR22"
 			(at 97.79 81.28 0)
 			(effects
@@
 			(project "DualCore6502Whole"
 				(path "/93e0914e-b2e9-49c2-95f2-7cc419f4ea20/578e6b65-8887-41c5-b062-8f45f343257b"
-					(reference "#PWR29")
+					(reference "#PWR22")
 					(unit 1)
 				)
@@
 		(dnp no)
 		(fields_autoplaced yes)
-		(property "Reference" "#PWR34"
+		(property "Reference" "#PWR27"
 			(at 149.86 143.51 0)
 			(effects
@@
 			(project "DualCore6502Whole"
 				(path "/93e0914e-b2e9-49c2-95f2-7cc419f4ea20/578e6b65-8887-41c5-b062-8f45f343257b"
-					(reference "#PWR34")
+					(reference "#PWR27")
 					(unit 1)
 				)
@@
 		(on_board yes)
 		(dnp no)
-		(property "Reference" "U4"
+		(property "Reference" "U3"
 			(at 156.21 58.42 0)
 			(effects
@@
 			(project "DualCore6502Whole"
 				(path "/93e0914e-b2e9-49c2-95f2-7cc419f4ea20/578e6b65-8887-41c5-b062-8f45f343257b"
-					(reference "U4")
+					(reference "U3")
 					(unit 1)
 				)
@@
 		(dnp no)
 		(fields_autoplaced yes)
-		(property "Reference" "C6"
+		(property "Reference" "C5"
 			(at 124.46 45.7199 0)
 			(effects
@@
 			(project "DualCore6502Whole"
 				(path "/93e0914e-b2e9-49c2-95f2-7cc419f4ea20/578e6b65-8887-41c5-b062-8f45f343257b"
-					(reference "C6")
+					(reference "C5")
 					(unit 1)
 				)

Commit message: Update the schematic
Parts:
- R8: value 33R -> 1K; footprint (none) -> Resistor_THT:R_Axial_DIN0207_L6.3mm_D2.5mm_P10.16mm_Horizontal
Connections:
- net CPU2_RDY is gone; now on net +5V: R8.1
Other:
- title: (none) -> Dual Core 65C02 Computer
Changed lines of the file:
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@@
 	(generator_version "8.0")
 	(paper "A4")
+	(title_block
+		(title "Dual Core 65C02 Computer")
+		(date "2026")
+		(comment 1 "Copyright (c) 2026 Rhys Weatherley")
+		(comment 3 "CPU 2")
+	)
 	(junction
 		(at 88.9 87.63)
@@
 		)
 	)
+	(wire
+		(pts
+			(xy 106.68 85.09) (xy 106.68 105.41)
+		)
+		(stroke
+			(width 0)
+			(type default)
+		)
+	)
 	(bus
 		(pts
@@
 		)
 	)
-	(wire
-		(pts
-			(xy 101.6 105.41) (xy 134.62 105.41)
-		)
-		(stroke
-			(width 0)
-			(type default)
-		)
-	)
 	(bus
 		(pts
@@
 		)
 	)
-	(wire
-		(pts
-			(xy 83.82 105.41) (xy 93.98 105.41)
-		)
-		(stroke
-			(width 0)
-			(type default)
-		)
-	)
 	(bus
 		(pts
@@
 		(pts
 			(xy 177.8 118.11) (xy 177.8 120.65)
+		)
+		(stroke
+			(width 0)
+			(type default)
+		)
+	)
+	(wire
+		(pts
+			(xy 106.68 105.41) (xy 134.62 105.41)
 		)
 		(stroke
@@
 		(property "Intersheetrefs" "${INTERSHEET_REFS}"
 			(at 114.2177 107.95 0)
-			(effects
-				(font
-					(size 1.27 1.27)
-				)
-				(justify right)
-				(hide yes)
-			)
-		)
-	)
-	(global_label "CPU2_RDY"
-		(shape input)
-		(at 83.82 105.41 180)
-		(fields_autoplaced yes)
-		(effects
-			(font
-				(size 1.27 1.27)
-			)
-			(justify right)
-		)
-		(property "Intersheetrefs" "${INTERSHEET_REFS}"
-			(at 71.1586 105.41 0)
 			(effects
 				(font
@@
 		(dnp no)
 		(fields_autoplaced yes)
-		(property "Reference" "#PWR23"
+		(property "Reference" "#PWR25"
 			(at 120.65 46.99 0)
 			(effects
@@
 			(project "DualCore6502Whole"
 				(path "/93e0914e-b2e9-49c2-95f2-7cc419f4ea20/578e6b65-8887-41c5-b062-8f45f343257b"
-					(reference "#PWR23")
+					(reference "#PWR25")
 					(unit 1)
 				)
@@
 		(dnp no)
 		(fields_autoplaced yes)
-		(property "Reference" "#PWR25"
+		(property "Reference" "#PWR27"
 			(at 133.35 128.27 0)
 			(effects
@@
 			(project "DualCore6502Whole"
 				(path "/93e0914e-b2e9-49c2-95f2-7cc419f4ea20/578e6b65-8887-41c5-b062-8f45f343257b"
-					(reference "#PWR25")
+					(reference "#PWR27")
 					(unit 1)
 				)
@@
 		(dnp no)
 		(fields_autoplaced yes)
-		(property "Reference" "#PWR21"
+		(property "Reference" "#PWR22"
 			(at 88.9 81.28 0)
 			(effects
@@
 			(project "DualCore6502Whole"
 				(path "/93e0914e-b2e9-49c2-95f2-7cc419f4ea20/578e6b65-8887-41c5-b062-8f45f343257b"
-					(reference "#PWR21")
+					(reference "#PWR22")
+					(unit 1)
+				)
+			)
+		)
+	)
+	(symbol
+		(lib_id "Device:R_US")
+		(at 106.68 81.28 0)
+		(unit 1)
+		(exclude_from_sim no)
+		(in_bom yes)
+		(on_board yes)
+		(dnp no)
+		(fields_autoplaced yes)
+		(property "Reference" "R8"
+			(at 109.22 80.0099 0)
+			(effects
+				(font
+					(size 1.27 1.27)
+				)
+				(justify left)
+			)
+		)
+		(property "Value" "1K"
+			(at 109.22 82.5499 0)
+			(effects
+				(font
+					(size 1.27 1.27)
+				)
+				(justify left)
+			)
+		)
+		(property "Footprint" "Resistor_THT:R_Axial_DIN0207_L6.3mm_D2.5mm_P10.16mm_Horizontal"
+			(at 107.696 81.534 90)
+			(effects
+				(font
+					(size 1.27 1.27)
+				)
+				(hide yes)
+			)
+		)
+		(property "Datasheet" "~"
+			(at 106.68 81.28 0)
+			(effects
+				(font
+					(size 1.27 1.27)
+				)
+				(hide yes)
+			)
+		)
+		(property "Description" "Resistor, US symbol"
+			(at 106.68 81.28 0)
+			(effects
+				(font
+					(size 1.27 1.27)
+				)
+				(hide yes)
+			)
+		)
+		(pin "2"
+		)
+		(pin "1"
+		)
+		(instances
+			(project "DualCore6502Whole"
+				(path "/93e0914e-b2e9-49c2-95f2-7cc419f4ea20/578e6b65-8887-41c5-b062-8f45f343257b"
+					(reference "R8")
 					(unit 1)
 				)
@@
 		(dnp no)
 		(fields_autoplaced yes)
-		(property "Reference" "#PWR24"
+		(property "Reference" "#PWR26"
 			(at 120.65 57.15 0)
 			(effects
@@
 		(property "Description" "Power symbol creates a global label with name \"GND\" , ground"
 			(at 120.65 50.8 0)
+			(effects
+				(font
+					(size 1.27 1.27)
+				)
+				(hide yes)
+			)
+		)
+		(pin "1"
+		)
+		(instances
+			(project "DualCore6502Whole"
+				(path "/93e0914e-b2e9-49c2-95f2-7cc419f4ea20/578e6b65-8887-41c5-b062-8f45f343257b"
+					(reference "#PWR26")
+					(unit 1)
+				)
+			)
+		)
+	)
+	(symbol
+		(lib_id "power:+5V")
+		(at 106.68 77.47 0)
+		(unit 1)
+		(exclude_from_sim no)
+		(in_bom yes)
+		(on_board yes)
+		(dnp no)
+		(fields_autoplaced yes)
+		(property "Reference" "#PWR24"
+			(at 106.68 81.28 0)
+			(effects
+				(font
+					(size 1.27 1.27)
+				)
+				(hide yes)
+			)
+		)
+		(property "Value" "+5V"
+			(at 106.68 72.39 0)
+			(effects
+				(font
+					(size 1.27 1.27)
+				)
+			)
+		)
+		(property "Footprint" ""
+			(at 106.68 77.47 0)
+			(effects
+				(font
+					(size 1.27 1.27)
+				)
+				(hide yes)
+			)
+		)
+		(property "Datasheet" ""
+			(at 106.68 77.47 0)
+			(effects
+				(font
+					(size 1.27 1.27)
+				)
+				(hide yes)
+			)
+		)
+		(property "Description" "Power symbol creates a global label with name \"+5V\""
+			(at 106.68 77.47 0)
 			(effects
 				(font
@@
 		(dnp no)
 		(fields_autoplaced yes)
-		(property "Reference" "#PWR26"
+		(property "Reference" "#PWR28"
 			(at 149.86 62.23 0)
 			(effects
@@
 			(project "DualCore6502Whole"
 				(path "/93e0914e-b2e9-49c2-95f2-7cc419f4ea20/578e6b65-8887-41c5-b062-8f45f343257b"
-					(reference "#PWR26")
+					(reference "#PWR28")
 					(unit 1)
 				)
@@
 		(dnp no)
 		(fields_autoplaced yes)
-		(property "Reference" "#PWR22"
+		(property "Reference" "#PWR23"
 			(at 97.79 81.28 0)
 			(effects
@@
 			(project "DualCore6502Whole"
 				(path "/93e0914e-b2e9-49c2-95f2-7cc419f4ea20/578e6b65-8887-41c5-b062-8f45f343257b"
-					(reference "#PWR22")
+					(reference "#PWR23")
 					(unit 1)
 				)
@@
 		(dnp no)
 		(fields_autoplaced yes)
-		(property "Reference" "#PWR27"
+		(property "Reference" "#PWR29"
 			(at 149.86 143.51 0)
 			(effects
@@
 			(project "DualCore6502Whole"
 				(path "/93e0914e-b2e9-49c2-95f2-7cc419f4ea20/578e6b65-8887-41c5-b062-8f45f343257b"
-					(reference "#PWR27")
+					(reference "#PWR29")
 					(unit 1)
 				)
@@
 					(unit 1)
 				)
-			)
-		)
-	)
-	(symbol
-		(lib_id "Device:R_US")
-		(at 97.79 105.41 90)
-		(unit 1)
-		(exclude_from_sim no)
-		(in_bom yes)
-		(on_board yes)
-		(dnp no)
-		(fields_autoplaced yes)
-		(property "Reference" "R8"
-			(at 97.79 99.06 90)
-			(effects
-				(font
-					(size 1.27 1.27)
-				)
-			)
-		)
-		(property "Value" "33R"
-			(at 97.79 101.6 90)
-			(effects
-				(font
-					(size 1.27 1.27)
-				)
-			)
-		)
-		(property "Footprint" ""
-			(at 98.044 104.394 90)
-			(effects
-				(font
-					(size 1.27 1.27)
-				)
-				(hide yes)
-			)
-		)
-		(property "Datasheet" "~"
-			(at 97.79 105.41 0)
-			(effects
-				(font
-					(size 1.27 1.27)
-				)
-				(hide yes)
-			)
-		)
-		(property "Description" "Resistor, US symbol"
-			(at 97.79 105.41 0)
-			(effects
-				(font
-					(size 1.27 1.27)
-				)
-				(hide yes)
-			)
-		)
-		(pin "1"
-		)
-		(pin "2"
-		)
-		(instances
-			(project "DualCore6502Whole"
-				(path "/93e0914e-b2e9-49c2-95f2-7cc419f4ea20/578e6b65-8887-41c5-b062-8f45f343257b"
-					(reference "R8")
-					(unit 1)
-				)

Commit message: Basic PCB layout
Parts:
- added TP4: CPU2 SYNC, TestPoint:TestPoint_Pad_D1.5mm, symbol Connector:TestPoint
- added TP5: ~{CPU2_VP}, TestPoint:TestPoint_Pad_D1.5mm, symbol Connector:TestPoint
- added TP6: ~{CPU2_ML}, TestPoint:TestPoint_Pad_D1.5mm, symbol Connector:TestPoint
- U2: renamed from U3; footprint Package_DIP:DIP-40_W15.24mm -> Package_DIP:DIP-40_W15.24mm_Socket
- renumbered C5 to C4
Connections:
- net CPU2_SYNC: no longer names the net of U2.7 (SYNC)
- net CPU2_SYNC: now also TP4.1
- net ~{CPU2_ML}: no longer names the net of U2.5 (~{ML})
- net ~{CPU2_ML}: now also TP6.1
- net ~{CPU2_VP}: no longer names the net of U2.1 (~{VP})
- net ~{CPU2_VP}: now also TP5.1
