File: schematics/DualCore6502Whole/memory.kicad_sch (KiCad schematic)
At the start: 6 parts, among them U10 62256, U11 28C256, U9 74HC86

Commit message: Remove the need to multiplex the control lines
Parts:
- renumbered C11 to C10, C12 to C11, C13 to C12, U11 to U10, U9 to U8, U10 to U9
Connections:
- net CPU_ID renamed CPU2_BUSEN
Changed lines of the file:
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@@
 		)
 	)
-	(global_label "CPU_ID"
+	(global_label "CPU2_BUSEN"
 		(shape input)
 		(at 74.93 114.3 180)
@@
 		)
 		(property "Intersheetrefs" "${INTERSHEET_REFS}"
-			(at 65.2319 114.3 0)
+			(at 59.6077 114.3 0)
 			(effects
 				(font
@@
 		)
 	)
-	(global_label "CPU_ID"
+	(global_label "CPU2_BUSEN"
 		(shape input)
 		(at 184.15 127 0)
@@
 		)
 		(property "Intersheetrefs" "${INTERSHEET_REFS}"
-			(at 193.8481 127 0)
+			(at 199.4723 127 0)
 			(effects
 				(font
@@
 		(dnp no)
 		(fields_autoplaced yes)
-		(property "Reference" "#PWR55"
+		(property "Reference" "#PWR48"
 			(at 35.56 180.34 0)
 			(effects
@@
 			(project "DualCore6502Whole"
 				(path "/93e0914e-b2e9-49c2-95f2-7cc419f4ea20/51d4148d-5301-42a5-a7b4-e8e185d89e40"
-					(reference "#PWR55")
+					(reference "#PWR48")
 					(unit 1)
 				)
@@
 		(dnp no)
 		(fields_autoplaced yes)
-		(property "Reference" "#PWR56"
+		(property "Reference" "#PWR49"
 			(at 53.34 55.88 0)
 			(effects
@@
 			(project "DualCore6502Whole"
 				(path "/93e0914e-b2e9-49c2-95f2-7cc419f4ea20/51d4148d-5301-42a5-a7b4-e8e185d89e40"
-					(reference "#PWR56")
+					(reference "#PWR49")
 					(unit 1)
 				)
@@
 		(dnp no)
 		(fields_autoplaced yes)
-		(property "Reference" "#PWR66"
+		(property "Reference" "#PWR59"
 			(at 166.37 148.59 0)
 			(effects
@@
 			(project "DualCore6502Whole"
 				(path "/93e0914e-b2e9-49c2-95f2-7cc419f4ea20/51d4148d-5301-42a5-a7b4-e8e185d89e40"
-					(reference "#PWR66")
+					(reference "#PWR59")
 					(unit 1)
 				)
@@
 		(dnp no)
 		(fields_autoplaced yes)
-		(property "Reference" "C13"
+		(property "Reference" "C12"
 			(at 186.69 68.58 0)
 			(effects
@@
 			(project "DualCore6502Whole"
 				(path "/93e0914e-b2e9-49c2-95f2-7cc419f4ea20/51d4148d-5301-42a5-a7b4-e8e185d89e40"
-					(reference "C13")
+					(reference "C12")
 					(unit 1)
 				)
@@
 		(dnp no)
 		(fields_autoplaced yes)
-		(property "Reference" "C12"
+		(property "Reference" "C11"
 			(at 91.44 158.75 0)
 			(effects
@@
 			(project "DualCore6502Whole"
 				(path "/93e0914e-b2e9-49c2-95f2-7cc419f4ea20/51d4148d-5301-42a5-a7b4-e8e185d89e40"
-					(reference "C12")
+					(reference "C11")
 					(unit 1)
 				)
@@
 		(dnp no)
 		(fields_autoplaced yes)
-		(property "Reference" "#PWR60"
+		(property "Reference" "#PWR53"
 			(at 87.63 160.02 0)
 			(effects
@@
 			(project "DualCore6502Whole"
 				(path "/93e0914e-b2e9-49c2-95f2-7cc419f4ea20/51d4148d-5301-42a5-a7b4-e8e185d89e40"
-					(reference "#PWR60")
+					(reference "#PWR53")
 					(unit 1)
 				)
@@
 		(dnp no)
 		(fields_autoplaced yes)
-		(property "Reference" "#PWR63"
+		(property "Reference" "#PWR56"
 			(at 113.03 107.95 0)
 			(effects
@@
 			(project "DualCore6502Whole"
 				(path "/93e0914e-b2e9-49c2-95f2-7cc419f4ea20/51d4148d-5301-42a5-a7b4-e8e185d89e40"
-					(reference "#PWR63")
+					(reference "#PWR56")
 					(unit 1)
 				)
@@
 		(dnp no)
 		(fields_autoplaced yes)
-		(property "Reference" "U11"
+		(property "Reference" "U10"
 			(at 169.3865 83.82 0)
 			(effects
@@
 			(project "DualCore6502Whole"
 				(path "/93e0914e-b2e9-49c2-95f2-7cc419f4ea20/51d4148d-5301-42a5-a7b4-e8e185d89e40"
-					(reference "U11")
+					(reference "U10")
 					(unit 1)
 				)
@@
 		(dnp no)
 		(fields_autoplaced yes)
-		(property "Reference" "#PWR58"
+		(property "Reference" "#PWR51"
 			(at 68.58 152.4 0)
 			(effects
@@
 			(project "DualCore6502Whole"
 				(path "/93e0914e-b2e9-49c2-95f2-7cc419f4ea20/51d4148d-5301-42a5-a7b4-e8e185d89e40"
-					(reference "#PWR58")
+					(reference "#PWR51")
 					(unit 1)
 				)
@@
 		(dnp no)
 		(fields_autoplaced yes)
-		(property "Reference" "#PWR70"
+		(property "Reference" "#PWR63"
 			(at 180.34 132.08 0)
 			(effects
@@
 			(project "DualCore6502Whole"
 				(path "/93e0914e-b2e9-49c2-95f2-7cc419f4ea20/51d4148d-5301-42a5-a7b4-e8e185d89e40"
-					(reference "#PWR70")
+					(reference "#PWR63")
 					(unit 1)
 				)
@@
 		(dnp no)
 		(fields_autoplaced yes)
-		(property "Reference" "#PWR62"
+		(property "Reference" "#PWR55"
 			(at 113.03 59.69 0)
 			(effects
@@
 			(project "DualCore6502Whole"
 				(path "/93e0914e-b2e9-49c2-95f2-7cc419f4ea20/51d4148d-5301-42a5-a7b4-e8e185d89e40"
-					(reference "#PWR62")
+					(reference "#PWR55")
 					(unit 1)
 				)
@@
 		(dnp no)
 		(fields_autoplaced yes)
-		(property "Reference" "#PWR68"
+		(property "Reference" "#PWR61"
 			(at 182.88 69.85 0)
 			(effects
@@
 			(project "DualCore6502Whole"
 				(path "/93e0914e-b2e9-49c2-95f2-7cc419f4ea20/51d4148d-5301-42a5-a7b4-e8e185d89e40"
-					(reference "#PWR68")
+					(reference "#PWR61")
 					(unit 1)
 				)
@@
 		(dnp no)
 		(fields_autoplaced yes)
-		(property "Reference" "U10"
+		(property "Reference" "U9"
 			(at 115.2241 53.34 0)
 			(effects
@@
 			(project "DualCore6502Whole"
 				(path "/93e0914e-b2e9-49c2-95f2-7cc419f4ea20/51d4148d-5301-42a5-a7b4-e8e185d89e40"
-					(reference "U10")
+					(reference "U9")
 					(unit 1)
 				)
@@
 		(dnp no)
 		(fields_autoplaced yes)
-		(property "Reference" "U9"
+		(property "Reference" "U8"
 			(at 45.4152 143.51 0)
 			(effects
@@
 			(project "DualCore6502Whole"
 				(path "/93e0914e-b2e9-49c2-95f2-7cc419f4ea20/51d4148d-5301-42a5-a7b4-e8e185d89e40"
-					(reference "U9")
+					(reference "U8")
 					(unit 2)
 				)
@@
 		(dnp no)
 		(fields_autoplaced yes)
-		(property "Reference" "#PWR69"
+		(property "Reference" "#PWR62"
 			(at 182.88 80.01 0)
 			(effects
@@
 			(project "DualCore6502Whole"
 				(path "/93e0914e-b2e9-49c2-95f2-7cc419f4ea20/51d4148d-5301-42a5-a7b4-e8e185d89e40"
-					(reference "#PWR69")
+					(reference "#PWR62")
 					(unit 1)
 				)
@@
 		(dnp no)
 		(fields_autoplaced yes)
-		(property "Reference" "#PWR59"
+		(property "Reference" "#PWR52"
 			(at 68.58 180.34 0)
 			(effects
@@
 			(project "DualCore6502Whole"
 				(path "/93e0914e-b2e9-49c2-95f2-7cc419f4ea20/51d4148d-5301-42a5-a7b4-e8e185d89e40"
-					(reference "#PWR59")
+					(reference "#PWR52")
 					(unit 1)
 				)
@@
 		(dnp no)
 		(fields_autoplaced yes)
-		(property "Reference" "#PWR67"
+		(property "Reference" "#PWR60"
 			(at 180.34 148.59 0)
 			(effects
@@
 			(project "DualCore6502Whole"
 				(path "/93e0914e-b2e9-49c2-95f2-7cc419f4ea20/51d4148d-5301-42a5-a7b4-e8e185d89e40"
-					(reference "#PWR67")
+					(reference "#PWR60")
 					(unit 1)
 				)
@@
 		(dnp no)
 		(fields_autoplaced yes)
-		(property "Reference" "U9"
+		(property "Reference" "U8"
 			(at 45.4152 127 0)
 			(effects
@@
 			(project "DualCore6502Whole"
 				(path "/93e0914e-b2e9-49c2-95f2-7cc419f4ea20/51d4148d-5301-42a5-a7b4-e8e185d89e40"
-					(reference "U9")
+					(reference "U8")
 					(unit 1)
 				)
@@
 		(dnp no)
 		(fields_autoplaced yes)
-		(property "Reference" "U9"
+		(property "Reference" "U8"
 			(at 74.93 160.0199 0)
 			(effects
@@
 			(project "DualCore6502Whole"
 				(path "/93e0914e-b2e9-49c2-95f2-7cc419f4ea20/51d4148d-5301-42a5-a7b4-e8e185d89e40"
-					(reference "U9")
+					(reference "U8")
 					(unit 5)
 				)
@@
 		(dnp no)
 		(fields_autoplaced yes)
-		(property "Reference" "U9"
+		(property "Reference" "U8"
 			(at 45.4152 160.02 0)
 			(effects
@@
 			(project "DualCore6502Whole"
 				(path "/93e0914e-b2e9-49c2-95f2-7cc419f4ea20/51d4148d-5301-42a5-a7b4-e8e185d89e40"
-					(reference "U9")
+					(reference "U8")
 					(unit 3)
 				)
@@
 		(dnp no)
 		(fields_autoplaced yes)
-		(property "Reference" "#PWR64"
+		(property "Reference" "#PWR57"
 			(at 137.16 100.33 0)
 			(effects
@@
 			(project "DualCore6502Whole"
 				(path "/93e0914e-b2e9-49c2-95f2-7cc419f4ea20/51d4148d-5301-42a5-a7b4-e8e185d89e40"
-					(reference "#PWR64")
+					(reference "#PWR57")
 					(unit 1)
 				)
@@
 		(dnp no)
 		(fields_autoplaced yes)
-		(property "Reference" "#PWR57"
+		(property "Reference" "#PWR50"
 			(at 53.34 66.04 0)
 			(effects
@@
 			(project "DualCore6502Whole"
 				(path "/93e0914e-b2e9-49c2-95f2-7cc419f4ea20/51d4148d-5301-42a5-a7b4-e8e185d89e40"
-					(reference "#PWR57")
+					(reference "#PWR50")
 					(unit 1)
 				)
@@
 		(dnp no)
 		(fields_autoplaced yes)
-		(property "Reference" "#PWR61"
+		(property "Reference" "#PWR54"
 			(at 87.63 170.18 0)
 			(effects
@@
 			(project "DualCore6502Whole"
 				(path "/93e0914e-b2e9-49c2-95f2-7cc419f4ea20/51d4148d-5301-42a5-a7b4-e8e185d89e40"
-					(reference "#PWR61")
+					(reference "#PWR54")
 					(unit 1)
 				)
@@
 		(dnp no)
 		(fields_autoplaced yes)
-		(property "Reference" "#PWR65"
+		(property "Reference" "#PWR58"
 			(at 166.37 90.17 0)
 			(effects
@@
 			(project "DualCore6502Whole"
 				(path "/93e0914e-b2e9-49c2-95f2-7cc419f4ea20/51d4148d-5301-42a5-a7b4-e8e185d89e40"
-					(reference "#PWR65")
+					(reference "#PWR58")
 					(unit 1)
 				)
@@
 		(dnp no)
 		(fields_autoplaced yes)
-		(property "Reference" "U9"
+		(property "Reference" "U8"
 			(at 88.5952 102.87 0)
 			(effects
@@
 			(project ""
 				(path "/93e0914e-b2e9-49c2-95f2-7cc419f4ea20/51d4148d-5301-42a5-a7b4-e8e185d89e40"
-					(reference "U9")
+					(reference "U8")
 					(unit 4)
 				)
@@
 		(dnp no)
 		(fields_autoplaced yes)
-		(property "Reference" "C11"
+		(property "Reference" "C10"
 			(at 57.15 54.61 0)
 			(effects
@@
 			(project "DualCore6502Whole"
 				(path "/93e0914e-b2e9-49c2-95f2-7cc419f4ea20/51d4148d-5301-42a5-a7b4-e8e185d89e40"
-					(reference "C11")
-					(unit 1)
-				)
+					(reference "C10")
+					(unit 1)
+				)

Commit message: Update the schematic
Parts:
- removed unit 2 of U8
- removed unit 1 of U8
- added C9: 100nF, Capacitor_THT:C_Disc_D5.0mm_W2.5mm_P5.00mm, symbol Device:C
- added U7: 74HC138, Package_DIP:DIP-16_W7.62mm, symbol 74xx:74LS138
Connections:
- net +5V: now also U8.10, C9.1, U7.16 (VCC)
- net A10: now also U7.1 (A0)
- net A11: now also U7.2 (A1)
- net A12: now also U7.3 (A2)
- net A13: now also U7.5 (E2)
- net A14: now also U9.1 (A14), U7.4 (E1); no longer U8.12
- net A9: now also U8.12; no longer U9.24 (A9)
- net CPU2_BUSEN: now also U7.6 (E3); no longer U8.13
- net GND: now also C9.2, U7.8 (GND); no longer U8.10, U8.9
- net at U8.11: now also U9.24 (A9); no longer U9.1 (A14)
- net at U8.8: now also U8.13
- new net: U7.15 (O0), U8.9
- no-connect marks 3 -> 7
Other:
- note added: "Shared 32K of RAM, $0000 to $7FFF. CPU2 swaps $0000 to $01FF with $0200 to $03FF to separate its zero page and stack from CPU1's."
- note removed: "Shared 32K of RAM, $0000 to $7FFF. CPU2 swaps the 16K halves to separate its zero page and stack from CPU1's."
- title: (none) -> Dual Core 65C02 Computer
- moved on the sheet: C10, C11, C12, U10, U8C, U8D, U8E, U9

Commit message: Update schematic and add 1ms NMI tick
Connections:
- net +5V: now also U8.13; no longer U8.10
- net A13: now also U7.4 (E1); no longer U7.5 (E2)
- net A14: now also U7.5 (E2); no longer U7.4 (E1)
- net A9: now also U8.9; no longer U8.12
- net at U7.15 (O0): now also U8.12; no longer U8.9
- net at U9.24 (A9): now also U8.8; no longer U8.11
- new net: U8.10, U8.11
Other:
- moved on the sheet: U8C, U8D

Commit message: Basic PCB layout
Parts:
- U6: renamed from U7; footprint Package_DIP:DIP-16_W7.62mm -> Package_DIP:DIP-16_W7.62mm_Socket
- U7: renamed from U8; footprint Package_DIP:DIP-14_W7.62mm -> Package_DIP:DIP-14_W7.62mm_Socket
- U8: renamed from U9; footprint Package_DIP:DIP-28_W15.24mm -> Package_DIP:DIP-28_W15.24mm_Socket
- renumbered C11 to C10, C12 to C11, C9 to C8, C10 to C9, U10 to U9
