File: schematics/DualCore6502Whole/mutex.kicad_sch (KiCad schematic)
At the start: 4 parts, among them U14 74HC374, U6 74HC02, U7 74HC32

Commit message: Remove the need to multiplex the control lines
Parts:
- renumbered C16 to C15, U14 to U13, U6 to U5, U7 to U6
Changed lines of the file:
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@@
 		(dnp no)
 		(fields_autoplaced yes)
-		(property "Reference" "U7"
+		(property "Reference" "U6"
 			(at 195.58 110.49 0)
 			(effects
@@
 			(project ""
 				(path "/93e0914e-b2e9-49c2-95f2-7cc419f4ea20/165c98f5-5fc6-4f55-a20e-8dbc47327a11"
-					(reference "U7")
+					(reference "U6")
 					(unit 3)
 				)
@@
 		(dnp no)
 		(fields_autoplaced yes)
-		(property "Reference" "U7"
+		(property "Reference" "U6"
 			(at 97.79 69.85 0)
 			(effects
@@
 			(project ""
 				(path "/93e0914e-b2e9-49c2-95f2-7cc419f4ea20/165c98f5-5fc6-4f55-a20e-8dbc47327a11"
-					(reference "U7")
+					(reference "U6")
 					(unit 1)
 				)
@@
 		(dnp no)
 		(fields_autoplaced yes)
-		(property "Reference" "U6"
+		(property "Reference" "U5"
 			(at 176.53 90.17 0)
 			(effects
@@
 			(project ""
 				(path "/93e0914e-b2e9-49c2-95f2-7cc419f4ea20/165c98f5-5fc6-4f55-a20e-8dbc47327a11"
-					(reference "U6")
+					(reference "U5")
 					(unit 3)
 				)
@@
 		(dnp no)
 		(fields_autoplaced yes)
-		(property "Reference" "U14"
+		(property "Reference" "U13"
 			(at 224.4441 68.58 0)
 			(effects
@@
 			(project ""
 				(path "/93e0914e-b2e9-49c2-95f2-7cc419f4ea20/165c98f5-5fc6-4f55-a20e-8dbc47327a11"
-					(reference "U14")
+					(reference "U13")
 					(unit 1)
 				)
@@
 		(dnp no)
 		(fields_autoplaced yes)
-		(property "Reference" "#PWR85"
+		(property "Reference" "#PWR78"
 			(at 222.25 142.24 0)
 			(effects
@@
 			(project "DualCore6502Whole"
 				(path "/93e0914e-b2e9-49c2-95f2-7cc419f4ea20/165c98f5-5fc6-4f55-a20e-8dbc47327a11"
-					(reference "#PWR85")
+					(reference "#PWR78")
 					(unit 1)
 				)
@@
 		(dnp no)
 		(fields_autoplaced yes)
-		(property "Reference" "#PWR84"
+		(property "Reference" "#PWR77"
 			(at 222.25 132.08 0)
 			(effects
@@
 			(project "DualCore6502Whole"
 				(path "/93e0914e-b2e9-49c2-95f2-7cc419f4ea20/165c98f5-5fc6-4f55-a20e-8dbc47327a11"
-					(reference "#PWR84")
+					(reference "#PWR77")
 					(unit 1)
 				)
@@
 		(dnp no)
 		(fields_autoplaced yes)
-		(property "Reference" "C16"
+		(property "Reference" "C15"
 			(at 226.06 130.81 0)
 			(effects
@@
 			(project "DualCore6502Whole"
 				(path "/93e0914e-b2e9-49c2-95f2-7cc419f4ea20/165c98f5-5fc6-4f55-a20e-8dbc47327a11"
-					(reference "C16")
+					(reference "C15")
 					(unit 1)
 				)
@@
 		(dnp no)
 		(fields_autoplaced yes)
-		(property "Reference" "#PWR83"
+		(property "Reference" "#PWR76"
 			(at 222.25 115.57 0)
 			(effects
@@
 			(project "DualCore6502Whole"
 				(path "/93e0914e-b2e9-49c2-95f2-7cc419f4ea20/165c98f5-5fc6-4f55-a20e-8dbc47327a11"
-					(reference "#PWR83")
+					(reference "#PWR76")
 					(unit 1)
 				)
@@
 		(dnp no)
 		(fields_autoplaced yes)
-		(property "Reference" "#PWR81"
+		(property "Reference" "#PWR74"
 			(at 163.83 133.35 0)
 			(effects
@@
 			(project ""
 				(path "/93e0914e-b2e9-49c2-95f2-7cc419f4ea20/165c98f5-5fc6-4f55-a20e-8dbc47327a11"
-					(reference "#PWR81")
+					(reference "#PWR74")
 					(unit 1)
 				)
@@
 		(dnp no)
 		(fields_autoplaced yes)
-		(property "Reference" "U7"
+		(property "Reference" "U6"
 			(at 97.79 87.63 0)
 			(effects
@@
 			(project ""
 				(path "/93e0914e-b2e9-49c2-95f2-7cc419f4ea20/165c98f5-5fc6-4f55-a20e-8dbc47327a11"
-					(reference "U7")
+					(reference "U6")
 					(unit 2)
 				)
@@
 		(dnp no)
 		(fields_autoplaced yes)
-		(property "Reference" "U6"
+		(property "Reference" "U5"
 			(at 176.53 113.03 0)
 			(effects
@@
 			(project ""
 				(path "/93e0914e-b2e9-49c2-95f2-7cc419f4ea20/165c98f5-5fc6-4f55-a20e-8dbc47327a11"
-					(reference "U6")
+					(reference "U5")
 					(unit 4)
 				)
@@
 		(dnp no)
 		(fields_autoplaced yes)
-		(property "Reference" "#PWR82"
+		(property "Reference" "#PWR75"
 			(at 222.25 72.39 0)
 			(effects
@@
 			(project ""
 				(path "/93e0914e-b2e9-49c2-95f2-7cc419f4ea20/165c98f5-5fc6-4f55-a20e-8dbc47327a11"
-					(reference "#PWR82")
+					(reference "#PWR75")
 					(unit 1)
 				)

Commit message: Add simpler I/O outputs as an alternative to the VIA
Parts:
- renumbered C15 to C16, U13 to U14
Changed lines of the file:
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@@
 		(dnp no)
 		(fields_autoplaced yes)
-		(property "Reference" "U13"
+		(property "Reference" "U14"
 			(at 224.4441 68.58 0)
 			(effects
@@
 			(project ""
 				(path "/93e0914e-b2e9-49c2-95f2-7cc419f4ea20/165c98f5-5fc6-4f55-a20e-8dbc47327a11"
-					(reference "U13")
+					(reference "U14")
 					(unit 1)
 				)
@@
 		(dnp no)
 		(fields_autoplaced yes)
-		(property "Reference" "#PWR78"
+		(property "Reference" "#PWR83"
 			(at 222.25 142.24 0)
 			(effects
@@
 			(project "DualCore6502Whole"
 				(path "/93e0914e-b2e9-49c2-95f2-7cc419f4ea20/165c98f5-5fc6-4f55-a20e-8dbc47327a11"
-					(reference "#PWR78")
+					(reference "#PWR83")
 					(unit 1)
 				)
@@
 		(dnp no)
 		(fields_autoplaced yes)
-		(property "Reference" "#PWR77"
+		(property "Reference" "#PWR82"
 			(at 222.25 132.08 0)
 			(effects
@@
 			(project "DualCore6502Whole"
 				(path "/93e0914e-b2e9-49c2-95f2-7cc419f4ea20/165c98f5-5fc6-4f55-a20e-8dbc47327a11"
-					(reference "#PWR77")
+					(reference "#PWR82")
 					(unit 1)
 				)
@@
 		(dnp no)
 		(fields_autoplaced yes)
-		(property "Reference" "C15"
+		(property "Reference" "C16"
 			(at 226.06 130.81 0)
 			(effects
@@
 			(project "DualCore6502Whole"
 				(path "/93e0914e-b2e9-49c2-95f2-7cc419f4ea20/165c98f5-5fc6-4f55-a20e-8dbc47327a11"
-					(reference "C15")
+					(reference "C16")
 					(unit 1)
 				)
@@
 		(dnp no)
 		(fields_autoplaced yes)
-		(property "Reference" "#PWR76"
+		(property "Reference" "#PWR81"
 			(at 222.25 115.57 0)
 			(effects
@@
 			(project "DualCore6502Whole"
 				(path "/93e0914e-b2e9-49c2-95f2-7cc419f4ea20/165c98f5-5fc6-4f55-a20e-8dbc47327a11"
-					(reference "#PWR76")
+					(reference "#PWR81")
 					(unit 1)
 				)
@@
 		(dnp no)
 		(fields_autoplaced yes)
-		(property "Reference" "#PWR74"
+		(property "Reference" "#PWR79"
 			(at 163.83 133.35 0)
 			(effects
@@
 			(project ""
 				(path "/93e0914e-b2e9-49c2-95f2-7cc419f4ea20/165c98f5-5fc6-4f55-a20e-8dbc47327a11"
-					(reference "#PWR74")
+					(reference "#PWR79")
 					(unit 1)
 				)
@@
 		(dnp no)
 		(fields_autoplaced yes)
-		(property "Reference" "#PWR75"
+		(property "Reference" "#PWR80"
 			(at 222.25 72.39 0)
 			(effects
@@
 			(project ""
 				(path "/93e0914e-b2e9-49c2-95f2-7cc419f4ea20/165c98f5-5fc6-4f55-a20e-8dbc47327a11"
-					(reference "#PWR75")
+					(reference "#PWR80")
 					(unit 1)
 				)

Commit message: Update the schematic
Parts:
- removed U14: 74HC374, Package_DIP:DIP-20_W7.62mm, symbol 74xx:74LS374
- removed U5: 74HC02, Package_DIP:DIP-14_W7.62mm, symbol 74xx:74LS02
- removed U6: 74HC32, Package_DIP:DIP-14_W7.62mm, symbol 74xx:74LS32
- added C15, C17, C18, C19, C20: 100nF, Capacitor_THT:C_Disc_D5.0mm_W2.5mm_P5.00mm, symbol Device:C
- added D3: IND4, LED_THT:LED_D3.0mm, symbol Device:LED
- added D4: IND3, LED_THT:LED_D3.0mm, symbol Device:LED
- added D5: IND2, LED_THT:LED_D3.0mm, symbol Device:LED
- added D6: IND1, LED_THT:LED_D3.0mm, symbol Device:LED
- added D7: IND0, LED_THT:LED_D3.0mm, symbol Device:LED
- added J3: Aux Inputs, Connector_PinHeader_2.54mm:PinHeader_2x05_P2.54mm_Vertical, symbol Connector_Generic:Conn_02x05_Odd_Even
- added R10, R11, R12, R13, R9: 470R, Resistor_THT:R_Axial_DIN0207_L6.3mm_D2.5mm_P10.16mm_Horizontal, symbol Device:R_US
- added U13: 74HC10, Package_DIP:DIP-14_W7.62mm, symbol 74xx:74LS10
- added U14: 74HC259, Package_DIP:DIP-16_W7.62mm, symbol 74xx:74LS259
- added U15: 74HC245, Package_DIP:DIP-20_W7.62mm, symbol 74xx:74HC245
- added U16: 74HC00, Package_DIP:DIP-14_W7.62mm, symbol 74xx:74LS00
- added U17: 74HC08, Package_DIP:DIP-14_W7.62mm, symbol 74xx:74LS08
- added U18: 74HC74, Package_DIP:DIP-14_W7.62mm, symbol 74xx:74LS74
Connections:
- net +5V: now also C15.1, C17.1, C18.1, C19.1, C20.1, U13.14 (VCC), U13.4, U13.5, U14.16 (VCC), U15.1 (A->B), U15.20 (VCC), U16.1, U16.10, U16.13, U16.14 (VCC), U16.2, U16.9, U17.14 (VCC), U18.10 (~{S}), U18.14 (VCC), U18.4 (~{S})
- net D0: now also U14.13 (D), U15.18 (B0)
- net D1: now also U15.17 (B1)
- net D2: now also U15.16 (B2)
- net D3: now also U15.15 (B3)
- net D4: now also U15.14 (B4)
- net D5: now also U15.13 (B5)
- net D6: now also U15.12 (B6)
- net D7: now also U15.11 (B7)
- net GND: now also C15.2, C17.2, C18.2, C19.2, C20.2, D3.1 (K), D4.1 (K), D5.1 (K), D6.1 (K), D7.1 (K), J3.1 (Pin_1), J3.3 (Pin_3), J3.5 (Pin_5), J3.7 (Pin_7), J3.9 (Pin_9), U13.7 (GND), U14.8 (GND), U15.10 (GND), U16.7 (GND), U17.10, U17.7 (GND), U17.9, U18.7 (GND)
- net ~{MUTEX_CS}: now also U13.3
- new net: U17.6, U18.11 (C)
- new net: U17.13, U18.8 (~{Q})
- new net: R12.1, U14.7 (Q3)
- new net: D4.2 (A), R12.2
- new net: D7.2 (A), R9.2
- new net: R10.1, U14.5 (Q1)
- new net: D6.2 (A), R10.2
- new net: U13.12, U15.19 (CE)
- new net: J3.2 (Pin_2), U15.2 (A0)
- new net: J3.4 (Pin_4), U15.3 (A1)
- new net: J3.6 (Pin_6), U15.4 (A2)
- new net: J3.8 (Pin_8), U15.5 (A3)
- new net: J3.10 (Pin_10), U15.6 (A4)
- new net: U17.11, U18.3 (C)
- new net: U16.6, U17.2
- new net: R13.1, U14.9 (Q4)
- new net: D3.2 (A), R13.2
- new net: R9.1, U14.4 (Q0)
- new net: D5.2 (A), R11.2
- new net: U13.10, U13.2, U13.6
- new net: U14.10 (Q5), U16.12
- new net: U13.8, U14.14 (E)
- new net: R11.1, U14.6 (Q2)
- new net: U17.1, U18.6 (~{Q})
- new net: U17.3, U17.4
- new net A0: U14.1 (A0)
- new net A1: U14.2 (A1)
- new net A2: U14.3 (A2)
- new net A7: U13.13
- new net A8: U13.11
- new net COMMON_CLK: U13.1, U13.9
- new net MAIN_CLK: U17.12, U17.5
- new net MUTEX_ACQ1: U15.9 (A7), U18.5 (Q)
- new net MUTEX_ACQ2: U15.8 (A6), U18.9 (Q)
- new net MUTEX_WANT1: U14.12 (Q7), U16.4, U18.2 (D)
- new net MUTEX_WANT2: U14.11 (Q6), U16.5, U18.12 (D)
- new net ~{CTS}: U15.7 (A5)
- new net ~{RESET}: U14.15 (Clr), U18.1 (~{R}), U18.13 (~{R})
- new net ~{RTS}: U16.11
- no-connect marks 0 -> 3
Other:
- note added: "Address range: $8100 to $8107, write-only"
- note added: "Address: $8080, read-only"
- note added: "To acquire the mutex, raise the MUTEX_WANTn line, then poll MUTEX_ACQn to wait for acquisition. To release the mutex, lower the MUTEX_WANTn line."
- note removed: "If a CPU is accessing the mutex counter for read-modify-write, disable the other CPU."
- note removed: "Mutex Counter"
- note removed: "mutex_init: lda #$ff sta $8000 rts mutex_lock: inc $8000 beq mutex_locked dec $8000 jmp mutex_lock mutex_locked: rts mutex_unlock: dec $8000 rts"
- title: (none) -> Dual Core 65C02 Computer

Commit message: Update schematic and add 1ms NMI tick
Connections:
- net +5V: now also U16.12, U16.4, U16.5; no longer U16.1, U16.10, U16.2
- net MUTEX_WANT1: now also U16.1; no longer U16.4
- net MUTEX_WANT2: now also U16.2; no longer U16.5
- net ~{RTS}: now also U16.8; no longer U16.11
- net at U16.6: no longer U17.2
- net at U14.10 (Q5): now also U16.10; no longer U16.12
- net at U16.3: now also U17.2
Other:
- moved on the sheet: U16A, U16B, U16C, U16D

Commit message: Basic PCB layout
Parts:
- U12: renamed from U13; footprint Package_DIP:DIP-14_W7.62mm -> Package_DIP:DIP-14_W7.62mm_Socket
- U13: renamed from U14; footprint Package_DIP:DIP-16_W7.62mm -> Package_DIP:DIP-16_W7.62mm_Socket
- U14: renamed from U15; footprint Package_DIP:DIP-20_W7.62mm -> Package_DIP:DIP-20_W7.62mm_Socket
- U15: renamed from U16; footprint Package_DIP:DIP-14_W7.62mm -> Package_DIP:DIP-14_W7.62mm_Socket
- U16: renamed from U17; footprint Package_DIP:DIP-14_W7.62mm -> Package_DIP:DIP-14_W7.62mm_Socket
- U17: renamed from U18; footprint Package_DIP:DIP-14_W7.62mm -> Package_DIP:DIP-14_W7.62mm_Socket
- renumbered C15 to C14, C16 to C15, C17 to C16, C18 to C17, C19 to C18, C20 to C19, D3 to D2, D4 to D3, D5 to D4, D6 to D5, D7 to D6
