File: schematics/DualCore6502Whole/rcbus.kicad_sch (KiCad schematic)
At the start: 8 parts, among them J5 Bus 1, U18 74HC00

Commit message: Remove the need to multiplex the control lines
Parts:
- renumbered C24 to C23, U18 to U17
Connections:
- net SYNC: no longer names the net of J5.47 (Pin_47)
- net ~{VP}: no longer names the net of J5.48 (Pin_48)
- no-connect marks 25 -> 27
Changed lines of the file:
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@@
 	)
 	(no_connect
+		(at 175.26 55.88)
+	)
+	(no_connect
 		(at 175.26 63.5)
 	)
@@
 	)
 	(no_connect
+		(at 175.26 58.42)
+	)
+	(no_connect
 		(at 175.26 106.68)
 	)
@@
 		)
 	)
-	(wire
-		(pts
-			(xy 175.26 55.88) (xy 179.07 55.88)
-		)
-		(stroke
-			(width 0)
-			(type default)
-		)
-	)
 	(bus
 		(pts
@@
 		)
 	)
-	(wire
-		(pts
-			(xy 175.26 58.42) (xy 179.07 58.42)
-		)
-		(stroke
-			(width 0)
-			(type default)
-		)
-	)
 	(bus
 		(pts
@@
 		)
 	)
-	(global_label "~{VP}"
-		(shape input)
-		(at 179.07 58.42 0)
-		(fields_autoplaced yes)
-		(effects
-			(font
-				(size 1.27 1.27)
-			)
-			(justify left)
-		)
-		(property "Intersheetrefs" "${INTERSHEET_REFS}"
-			(at 184.4138 58.42 0)
-			(effects
-				(font
-					(size 1.27 1.27)
-				)
-				(justify left)
-				(hide yes)
-			)
-		)
-	)
 	(global_label "~{CPU1_NMI}"
 		(shape output)
@@
 		)
 	)
-	(global_label "SYNC"
-		(shape input)
-		(at 179.07 55.88 0)
-		(fields_autoplaced yes)
-		(effects
-			(font
-				(size 1.27 1.27)
-			)
-			(justify left)
-		)
-		(property "Intersheetrefs" "${INTERSHEET_REFS}"
-			(at 186.9538 55.88 0)
-			(effects
-				(font
-					(size 1.27 1.27)
-				)
-				(justify left)
-				(hide yes)
-			)
-		)
-	)
 	(global_label "~{MEMRQ}"
 		(shape output)
@@
 		(dnp no)
 		(fields_autoplaced yes)
-		(property "Reference" "#PWR109"
+		(property "Reference" "#PWR102"
 			(at 151.13 81.28 0)
 			(effects
@@
 			(project "DualCore6502Whole"
 				(path "/93e0914e-b2e9-49c2-95f2-7cc419f4ea20/3412cf2c-7ca6-479d-a9c2-89b197305d30"
-					(reference "#PWR109")
+					(reference "#PWR102")
 					(unit 1)
 				)
@@
 		(dnp no)
 		(fields_autoplaced yes)
-		(property "Reference" "#PWR104"
+		(property "Reference" "#PWR97"
 			(at 43.18 191.77 0)
 			(effects
@@
 			(project "DualCore6502Whole"
 				(path "/93e0914e-b2e9-49c2-95f2-7cc419f4ea20/3412cf2c-7ca6-479d-a9c2-89b197305d30"
-					(reference "#PWR104")
+					(reference "#PWR97")
 					(unit 1)
 				)
@@
 		(dnp no)
 		(fields_autoplaced yes)
-		(property "Reference" "C24"
+		(property "Reference" "C23"
 			(at 68.58 171.45 0)
 			(effects
@@
 			(project "DualCore6502Whole"
 				(path "/93e0914e-b2e9-49c2-95f2-7cc419f4ea20/3412cf2c-7ca6-479d-a9c2-89b197305d30"
-					(reference "C24")
+					(reference "C23")
 					(unit 1)
 				)
@@
 		(dnp no)
 		(fields_autoplaced yes)
-		(property "Reference" "U18"
+		(property "Reference" "U17"
 			(at 99.0517 111.76 0)
 			(effects
@@
 			(project ""
 				(path "/93e0914e-b2e9-49c2-95f2-7cc419f4ea20/3412cf2c-7ca6-479d-a9c2-89b197305d30"
-					(reference "U18")
+					(reference "U17")
 					(unit 3)
 				)
@@
 		(dnp no)
 		(fields_autoplaced yes)
-		(property "Reference" "U18"
+		(property "Reference" "U17"
 			(at 77.4617 71.12 0)
 			(effects
@@
 			(project ""
 				(path "/93e0914e-b2e9-49c2-95f2-7cc419f4ea20/3412cf2c-7ca6-479d-a9c2-89b197305d30"
-					(reference "U18")
+					(reference "U17")
 					(unit 1)
 				)
@@
 		(dnp no)
 		(fields_autoplaced yes)
-		(property "Reference" "#PWR116"
+		(property "Reference" "#PWR109"
 			(at 231.14 81.28 0)
 			(effects
@@
 			(project "DualCore6502Whole"
 				(path "/93e0914e-b2e9-49c2-95f2-7cc419f4ea20/3412cf2c-7ca6-479d-a9c2-89b197305d30"
-					(reference "#PWR116")
+					(reference "#PWR109")
 					(unit 1)
 				)
@@
 		(dnp no)
 		(fields_autoplaced yes)
-		(property "Reference" "#PWR110"
+		(property "Reference" "#PWR103"
 			(at 161.29 83.82 0)
 			(effects
@@
 			(project "DualCore6502Whole"
 				(path "/93e0914e-b2e9-49c2-95f2-7cc419f4ea20/3412cf2c-7ca6-479d-a9c2-89b197305d30"
-					(reference "#PWR110")
+					(reference "#PWR103")
 					(unit 1)
 				)
@@
 		(dnp no)
 		(fields_autoplaced yes)
-		(property "Reference" "U18"
+		(property "Reference" "U17"
 			(at 50.8 171.4499 0)
 			(effects
@@
 			(project ""
 				(path "/93e0914e-b2e9-49c2-95f2-7cc419f4ea20/3412cf2c-7ca6-479d-a9c2-89b197305d30"
-					(reference "U18")
+					(reference "U17")
 					(unit 5)
 				)
@@
 		(dnp no)
 		(fields_autoplaced yes)
-		(property "Reference" "U18"
+		(property "Reference" "U17"
 			(at 77.4617 90.17 0)
 			(effects
@@
 			(project ""
 				(path "/93e0914e-b2e9-49c2-95f2-7cc419f4ea20/3412cf2c-7ca6-479d-a9c2-89b197305d30"
-					(reference "U18")
+					(reference "U17")
 					(unit 2)
 				)
@@
 		(dnp no)
 		(fields_autoplaced yes)
-		(property "Reference" "#PWR107"
+		(property "Reference" "#PWR100"
 			(at 64.77 182.88 0)
 			(effects
@@
 			(project "DualCore6502Whole"
 				(path "/93e0914e-b2e9-49c2-95f2-7cc419f4ea20/3412cf2c-7ca6-479d-a9c2-89b197305d30"
-					(reference "#PWR107")
+					(reference "#PWR100")
 					(unit 1)
 				)
@@
 		(dnp no)
 		(fields_autoplaced yes)
-		(property "Reference" "#PWR106"
+		(property "Reference" "#PWR99"
 			(at 64.77 172.72 0)
 			(effects
@@
 			(project "DualCore6502Whole"
 				(path "/93e0914e-b2e9-49c2-95f2-7cc419f4ea20/3412cf2c-7ca6-479d-a9c2-89b197305d30"
-					(reference "#PWR106")
+					(reference "#PWR99")
 					(unit 1)
 				)
@@
 		(dnp no)
 		(fields_autoplaced yes)
-		(property "Reference" "U18"
+		(property "Reference" "U17"
 			(at 77.4617 109.22 0)
 			(effects
@@
 			(project ""
 				(path "/93e0914e-b2e9-49c2-95f2-7cc419f4ea20/3412cf2c-7ca6-479d-a9c2-89b197305d30"
-					(reference "U18")
+					(reference "U17")
 					(unit 4)
 				)
@@
 		(dnp no)
 		(fields_autoplaced yes)
-		(property "Reference" "#PWR111"
+		(property "Reference" "#PWR104"
 			(at 186.69 81.28 0)
 			(effects
@@
 			(project "DualCore6502Whole"
 				(path "/93e0914e-b2e9-49c2-95f2-7cc419f4ea20/3412cf2c-7ca6-479d-a9c2-89b197305d30"
-					(reference "#PWR111")
+					(reference "#PWR104")
 					(unit 1)
 				)
@@
 		(dnp no)
 		(fields_autoplaced yes)
-		(property "Reference" "#PWR113"
+		(property "Reference" "#PWR106"
 			(at 200.66 81.28 0)
 			(effects
@@
 			(project "DualCore6502Whole"
 				(path "/93e0914e-b2e9-49c2-95f2-7cc419f4ea20/3412cf2c-7ca6-479d-a9c2-89b197305d30"
-					(reference "#PWR113")
+					(reference "#PWR106")
 					(unit 1)
 				)
@@
 		(dnp no)
 		(fields_autoplaced yes)
-		(property "Reference" "#PWR108"
+		(property "Reference" "#PWR101"
 			(at 135.89 81.28 0)
 			(effects
@@
 			(project "DualCore6502Whole"
 				(path "/93e0914e-b2e9-49c2-95f2-7cc419f4ea20/3412cf2c-7ca6-479d-a9c2-89b197305d30"
-					(reference "#PWR108")
+					(reference "#PWR101")
 					(unit 1)
 				)
@@
 		(dnp no)
 		(fields_autoplaced yes)
-		(property "Reference" "#PWR115"
+		(property "Reference" "#PWR108"
 			(at 220.98 81.28 0)
 			(effects
@@
 			(project "DualCore6502Whole"
 				(path "/93e0914e-b2e9-49c2-95f2-7cc419f4ea20/3412cf2c-7ca6-479d-a9c2-89b197305d30"
-					(reference "#PWR115")
+					(reference "#PWR108")
 					(unit 1)
 				)
@@
 		(dnp no)
 		(fields_autoplaced yes)
-		(property "Reference" "#PWR105"
+		(property "Reference" "#PWR98"
 			(at 62.23 78.74 0)
 			(effects
@@
 			(project "DualCore6502Whole"
 				(path "/93e0914e-b2e9-49c2-95f2-7cc419f4ea20/3412cf2c-7ca6-479d-a9c2-89b197305d30"
-					(reference "#PWR105")
+					(reference "#PWR98")
 					(unit 1)
 				)
@@
 		(dnp no)
 		(fields_autoplaced yes)
-		(property "Reference" "#PWR103"
+		(property "Reference" "#PWR96"
 			(at 43.18 163.83 0)
 			(effects
@@
 			(project "DualCore6502Whole"
 				(path "/93e0914e-b2e9-49c2-95f2-7cc419f4ea20/3412cf2c-7ca6-479d-a9c2-89b197305d30"
-					(reference "#PWR103")
+					(reference "#PWR96")
 					(unit 1)
 				)
@@
 		(dnp no)
 		(fields_autoplaced yes)
-		(property "Reference" "#PWR114"
+		(property "Reference" "#PWR107"
 			(at 210.82 81.28 0)
 			(effects
@@
 			(project "DualCore6502Whole"
 				(path "/93e0914e-b2e9-49c2-95f2-7cc419f4ea20/3412cf2c-7ca6-479d-a9c2-89b197305d30"
-					(reference "#PWR114")
+					(reference "#PWR107")
 					(unit 1)
 				)
@@
 		(dnp no)
 		(fields_autoplaced yes)
-		(property "Reference" "#PWR112"
+		(property "Reference" "#PWR105"
 			(at 176.53 83.82 0)
 			(effects
@@
 			(project "DualCore6502Whole"
 				(path "/93e0914e-b2e9-49c2-95f2-7cc419f4ea20/3412cf2c-7ca6-479d-a9c2-89b197305d30"
-					(reference "#PWR112")
+					(reference "#PWR105")
 					(unit 1)
 				)

Commit message: Add simpler I/O outputs as an alternative to the VIA
Parts:
- renumbered C23 to C25, J5 to J6, U17 to U19
Connections:
- net +5V: now also U19.13
- net R/~{W}: no longer U19.13
Changed lines of the file:
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@@
 		(color 0 0 0 0)
 	)
-	(junction
-		(at 67.31 115.57)
-		(diameter 0)
-		(color 0 0 0 0)
-	)
 	(no_connect
 		(at 175.26 73.66)
@@
 	(wire
 		(pts
-			(xy 69.85 120.65) (xy 67.31 120.65)
-		)
-		(stroke
-			(width 0)
-			(type default)
-		)
-	)
-	(wire
-		(pts
 			(xy 175.26 50.8) (xy 179.07 50.8)
 		)
@@
 	(wire
 		(pts
-			(xy 67.31 120.65) (xy 67.31 115.57)
+			(xy 64.77 120.65) (xy 69.85 120.65)
 		)
 		(stroke
@@
 		(dnp no)
 		(fields_autoplaced yes)
-		(property "Reference" "J5"
+		(property "Reference" "J6"
 			(at 168.91 34.29 0)
 			(effects
@@
 			(project "DualCore6502Whole"
 				(path "/93e0914e-b2e9-49c2-95f2-7cc419f4ea20/3412cf2c-7ca6-479d-a9c2-89b197305d30"
-					(reference "J5")
+					(reference "J6")
 					(unit 1)
 				)
@@
 		(dnp no)
 		(fields_autoplaced yes)
-		(property "Reference" "#PWR102"
+		(property "Reference" "#PWR112"
 			(at 151.13 81.28 0)
 			(effects
@@
 			(project "DualCore6502Whole"
 				(path "/93e0914e-b2e9-49c2-95f2-7cc419f4ea20/3412cf2c-7ca6-479d-a9c2-89b197305d30"
-					(reference "#PWR102")
+					(reference "#PWR112")
 					(unit 1)
 				)
@@
 		(dnp no)
 		(fields_autoplaced yes)
-		(property "Reference" "#PWR97"
+		(property "Reference" "#PWR107"
 			(at 43.18 191.77 0)
 			(effects
@@
 			(project "DualCore6502Whole"
 				(path "/93e0914e-b2e9-49c2-95f2-7cc419f4ea20/3412cf2c-7ca6-479d-a9c2-89b197305d30"
-					(reference "#PWR97")
+					(reference "#PWR107")
 					(unit 1)
 				)
@@
 		(dnp no)
 		(fields_autoplaced yes)
-		(property "Reference" "C23"
+		(property "Reference" "C25"
 			(at 68.58 171.45 0)
 			(effects
@@
 			(project "DualCore6502Whole"
 				(path "/93e0914e-b2e9-49c2-95f2-7cc419f4ea20/3412cf2c-7ca6-479d-a9c2-89b197305d30"
-					(reference "C23")
+					(reference "C25")
 					(unit 1)
 				)
@@
 		(dnp no)
 		(fields_autoplaced yes)
-		(property "Reference" "U17"
+		(property "Reference" "U19"
 			(at 99.0517 111.76 0)
 			(effects
@@
 			(project ""
 				(path "/93e0914e-b2e9-49c2-95f2-7cc419f4ea20/3412cf2c-7ca6-479d-a9c2-89b197305d30"
-					(reference "U17")
+					(reference "U19")
 					(unit 3)
 				)
@@
 		(dnp no)
 		(fields_autoplaced yes)
-		(property "Reference" "U17"
+		(property "Reference" "U19"
 			(at 77.4617 71.12 0)
 			(effects
@@
 			(project ""
 				(path "/93e0914e-b2e9-49c2-95f2-7cc419f4ea20/3412cf2c-7ca6-479d-a9c2-89b197305d30"
-					(reference "U17")
+					(reference "U19")
 					(unit 1)
 				)
@@
 		(dnp no)
 		(fields_autoplaced yes)
-		(property "Reference" "#PWR109"
+		(property "Reference" "#PWR119"
 			(at 231.14 81.28 0)
 			(effects
@@
 			(project "DualCore6502Whole"
 				(path "/93e0914e-b2e9-49c2-95f2-7cc419f4ea20/3412cf2c-7ca6-479d-a9c2-89b197305d30"
-					(reference "#PWR109")
+					(reference "#PWR119")
 					(unit 1)
 				)
@@
 		(dnp no)
 		(fields_autoplaced yes)
-		(property "Reference" "#PWR103"
+		(property "Reference" "#PWR113"
 			(at 161.29 83.82 0)
 			(effects
@@
 			(project "DualCore6502Whole"
 				(path "/93e0914e-b2e9-49c2-95f2-7cc419f4ea20/3412cf2c-7ca6-479d-a9c2-89b197305d30"
-					(reference "#PWR103")
+					(reference "#PWR113")
 					(unit 1)
 				)
@@
 		(dnp no)
 		(fields_autoplaced yes)
-		(property "Reference" "U17"
+		(property "Reference" "U19"
 			(at 50.8 171.4499 0)
 			(effects
@@
 			(project ""
 				(path "/93e0914e-b2e9-49c2-95f2-7cc419f4ea20/3412cf2c-7ca6-479d-a9c2-89b197305d30"
-					(reference "U17")
+					(reference "U19")
 					(unit 5)
 				)
@@
 		(dnp no)
 		(fields_autoplaced yes)
-		(property "Reference" "U17"
+		(property "Reference" "U19"
 			(at 77.4617 90.17 0)
 			(effects
@@
 			(project ""
 				(path "/93e0914e-b2e9-49c2-95f2-7cc419f4ea20/3412cf2c-7ca6-479d-a9c2-89b197305d30"
-					(reference "U17")
+					(reference "U19")
 					(unit 2)
 				)
@@
 		(dnp no)
 		(fields_autoplaced yes)
-		(property "Reference" "#PWR100"
+		(property "Reference" "#PWR110"
 			(at 64.77 182.88 0)
 			(effects
@@
 			(project "DualCore6502Whole"
 				(path "/93e0914e-b2e9-49c2-95f2-7cc419f4ea20/3412cf2c-7ca6-479d-a9c2-89b197305d30"
-					(reference "#PWR100")
+					(reference "#PWR110")
 					(unit 1)
 				)
@@
 		(dnp no)
 		(fields_autoplaced yes)
-		(property "Reference" "#PWR99"
+		(property "Reference" "#PWR109"
 			(at 64.77 172.72 0)
 			(effects
@@
 			(project "DualCore6502Whole"
 				(path "/93e0914e-b2e9-49c2-95f2-7cc419f4ea20/3412cf2c-7ca6-479d-a9c2-89b197305d30"
-					(reference "#PWR99")
+					(reference "#PWR109")
 					(unit 1)
 				)
@@
 		(dnp no)
 		(fields_autoplaced yes)
-		(property "Reference" "U17"
+		(property "Reference" "U19"
 			(at 77.4617 109.22 0)
 			(effects
@@
 			(project ""
 				(path "/93e0914e-b2e9-49c2-95f2-7cc419f4ea20/3412cf2c-7ca6-479d-a9c2-89b197305d30"
-					(reference "U17")
+					(reference "U19")
 					(unit 4)
 				)
@@
 		(dnp no)
 		(fields_autoplaced yes)
-		(property "Reference" "#PWR104"
+		(property "Reference" "#PWR114"
 			(at 186.69 81.28 0)
 			(effects
@@
 			(project "DualCore6502Whole"
 				(path "/93e0914e-b2e9-49c2-95f2-7cc419f4ea20/3412cf2c-7ca6-479d-a9c2-89b197305d30"
-					(reference "#PWR104")
+					(reference "#PWR114")
 					(unit 1)
 				)
@@
 		(dnp no)
 		(fields_autoplaced yes)
-		(property "Reference" "#PWR106"
+		(property "Reference" "#PWR116"
 			(at 200.66 81.28 0)
 			(effects
@@
 			(project "DualCore6502Whole"
 				(path "/93e0914e-b2e9-49c2-95f2-7cc419f4ea20/3412cf2c-7ca6-479d-a9c2-89b197305d30"
-					(reference "#PWR106")
+					(reference "#PWR116")
 					(unit 1)
 				)
@@
 		(dnp no)
 		(fields_autoplaced yes)
-		(property "Reference" "#PWR101"
+		(property "Reference" "#PWR111"
 			(at 135.89 81.28 0)
 			(effects
@@
 			(project "DualCore6502Whole"
 				(path "/93e0914e-b2e9-49c2-95f2-7cc419f4ea20/3412cf2c-7ca6-479d-a9c2-89b197305d30"
-					(reference "#PWR101")
+					(reference "#PWR111")
 					(unit 1)
 				)
@@
 		(dnp no)
 		(fields_autoplaced yes)
-		(property "Reference" "#PWR108"
+		(property "Reference" "#PWR118"
 			(at 220.98 81.28 0)
 			(effects
@@
 			(project "DualCore6502Whole"
 				(path "/93e0914e-b2e9-49c2-95f2-7cc419f4ea20/3412cf2c-7ca6-479d-a9c2-89b197305d30"
-					(reference "#PWR108")
+					(reference "#PWR118")
 					(unit 1)
 				)
@@
 		(dnp no)
 		(fields_autoplaced yes)
-		(property "Reference" "#PWR98"
+		(property "Reference" "#PWR108"
 			(at 62.23 78.74 0)
 			(effects
@@
 			(project "DualCore6502Whole"
 				(path "/93e0914e-b2e9-49c2-95f2-7cc419f4ea20/3412cf2c-7ca6-479d-a9c2-89b197305d30"
-					(reference "#PWR98")
+					(reference "#PWR108")
 					(unit 1)
 				)
@@
 		(dnp no)
 		(fields_autoplaced yes)
-		(property "Reference" "#PWR96"
+		(property "Reference" "#PWR106"
 			(at 43.18 163.83 0)
 			(effects
@@
 			(project "DualCore6502Whole"
 				(path "/93e0914e-b2e9-49c2-95f2-7cc419f4ea20/3412cf2c-7ca6-479d-a9c2-89b197305d30"
-					(reference "#PWR96")
+					(reference "#PWR106")
+					(unit 1)
+				)
+			)
+		)
+	)
+	(symbol
+		(lib_id "power:+5V")
+		(at 64.77 120.65 90)
+		(unit 1)
+		(exclude_from_sim no)
+		(in_bom yes)
+		(on_board yes)
+		(dnp no)
+		(fields_autoplaced yes)
+		(property "Reference" "#PWR120"
+			(at 68.58 120.65 0)
+			(effects
+				(font
+					(size 1.27 1.27)
+				)
+				(hide yes)
+			)
+		)
+		(property "Value" "+5V"
+			(at 60.96 120.6499 90)
+			(effects
+				(font
+					(size 1.27 1.27)
+				)
+				(justify left)
+			)
+		)
+		(property "Footprint" ""
+			(at 64.77 120.65 0)
+			(effects
+				(font
+					(size 1.27 1.27)
+				)
+				(hide yes)
+			)
+		)
+		(property "Datasheet" ""
+			(at 64.77 120.65 0)
+			(effects
+				(font
+					(size 1.27 1.27)
+				)
+				(hide yes)
+			)
+		)
+		(property "Description" "Power symbol creates a global label with name \"+5V\""
+			(at 64.77 120.65 0)
+			(effects
+				(font
+					(size 1.27 1.27)
+				)
+				(hide yes)
+			)
+		)
+		(pin "1"
+		)
+		(instances
+			(project "DualCore6502Whole"
+				(path "/93e0914e-b2e9-49c2-95f2-7cc419f4ea20/3412cf2c-7ca6-479d-a9c2-89b197305d30"
+					(reference "#PWR120")
 					(unit 1)
 				)
@@
 		(dnp no)
 		(fields_autoplaced yes)
-		(property "Reference" "#PWR107"
+		(property "Reference" "#PWR117"
 			(at 210.82 81.28 0)
 			(effects
@@
 			(project "DualCore6502Whole"
 				(path "/93e0914e-b2e9-49c2-95f2-7cc419f4ea20/3412cf2c-7ca6-479d-a9c2-89b197305d30"
-					(reference "#PWR107")
+					(reference "#PWR117")
 					(unit 1)
 				)
@@
 		(dnp no)
 		(fields_autoplaced yes)
-		(property "Reference" "#PWR105"
+		(property "Reference" "#PWR115"
 			(at 176.53 83.82 0)
 			(effects
@@
 			(project "DualCore6502Whole"
 				(path "/93e0914e-b2e9-49c2-95f2-7cc419f4ea20/3412cf2c-7ca6-479d-a9c2-89b197305d30"
-					(reference "#PWR105")
+					(reference "#PWR115")
 					(unit 1)
 				)
