File: schematics/DualCore6502Whole/rcbus.kicad_sch (KiCad schematic)
At the start: 8 parts, among them J6 Bus 1, U19 74HC00

Commit message: Update the schematic
Parts:
- renumbered C25 to C28, R10 to R15, R11 to R16, R12 to R17, R13 to R18, R14 to R19, U19 to U22
Other:
- title: (none) -> Dual Core 65C02 Computer
Changed lines of the file:
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@@
 	(generator_version "8.0")
 	(paper "A4")
+	(title_block
+		(title "Dual Core 65C02 Computer")
+		(date "2026")
+		(comment 1 "Copyright (c) 2026 Rhys Weatherley")
+		(comment 3 "RCBus Interface")
+	)
 	(junction
 		(at 67.31 101.6)
@@
 		(dnp no)
 		(fields_autoplaced yes)
-		(property "Reference" "#PWR112"
+		(property "Reference" "#PWR141"
 			(at 151.13 81.28 0)
 			(effects
@@
 			(project "DualCore6502Whole"
 				(path "/93e0914e-b2e9-49c2-95f2-7cc419f4ea20/3412cf2c-7ca6-479d-a9c2-89b197305d30"
-					(reference "#PWR112")
+					(reference "#PWR141")
 					(unit 1)
 				)
@@
 		(dnp no)
 		(fields_autoplaced yes)
-		(property "Reference" "#PWR107"
+		(property "Reference" "#PWR135"
 			(at 43.18 191.77 0)
 			(effects
@@
 			(project "DualCore6502Whole"
 				(path "/93e0914e-b2e9-49c2-95f2-7cc419f4ea20/3412cf2c-7ca6-479d-a9c2-89b197305d30"
-					(reference "#PWR107")
+					(reference "#PWR135")
 					(unit 1)
 				)
@@
 		(dnp no)
 		(fields_autoplaced yes)
-		(property "Reference" "C25"
+		(property "Reference" "C28"
 			(at 68.58 171.45 0)
 			(effects
@@
 			(project "DualCore6502Whole"
 				(path "/93e0914e-b2e9-49c2-95f2-7cc419f4ea20/3412cf2c-7ca6-479d-a9c2-89b197305d30"
-					(reference "C25")
+					(reference "C28")
 					(unit 1)
 				)
@@
 		(on_board yes)
 		(dnp no)
-		(property "Reference" "R11"
+		(property "Reference" "R16"
 			(at 203.2 80.0099 0)
 			(effects
@@
 			(project "DualCore6502Whole"
 				(path "/93e0914e-b2e9-49c2-95f2-7cc419f4ea20/3412cf2c-7ca6-479d-a9c2-89b197305d30"
-					(reference "R11")
+					(reference "R16")
 					(unit 1)
 				)
@@
 		(on_board yes)
 		(dnp no)
-		(property "Reference" "R10"
+		(property "Reference" "R15"
 			(at 133.35 80.0099 0)
 			(effects
@@
 			(project "DualCore6502Whole"
 				(path "/93e0914e-b2e9-49c2-95f2-7cc419f4ea20/3412cf2c-7ca6-479d-a9c2-89b197305d30"
-					(reference "R10")
+					(reference "R15")
 					(unit 1)
 				)
@@
 		(dnp no)
 		(fields_autoplaced yes)
-		(property "Reference" "U19"
+		(property "Reference" "U22"
 			(at 99.0517 111.76 0)
 			(effects
@@
 			(project ""
 				(path "/93e0914e-b2e9-49c2-95f2-7cc419f4ea20/3412cf2c-7ca6-479d-a9c2-89b197305d30"
-					(reference "U19")
+					(reference "U22")
 					(unit 3)
 				)
@@
 		(dnp no)
 		(fields_autoplaced yes)
-		(property "Reference" "U19"
+		(property "Reference" "U22"
 			(at 77.4617 71.12 0)
 			(effects
@@
 			(project ""
 				(path "/93e0914e-b2e9-49c2-95f2-7cc419f4ea20/3412cf2c-7ca6-479d-a9c2-89b197305d30"
-					(reference "U19")
+					(reference "U22")
 					(unit 1)
 				)
@@
 		(on_board yes)
 		(dnp no)
-		(property "Reference" "R13"
+		(property "Reference" "R18"
 			(at 223.52 80.0099 0)
 			(effects
@@
 			(project "DualCore6502Whole"
 				(path "/93e0914e-b2e9-49c2-95f2-7cc419f4ea20/3412cf2c-7ca6-479d-a9c2-89b197305d30"
-					(reference "R13")
+					(reference "R18")
 					(unit 1)
 				)
@@
 		(dnp no)
 		(fields_autoplaced yes)
-		(property "Reference" "#PWR119"
+		(property "Reference" "#PWR148"
 			(at 231.14 81.28 0)
 			(effects
@@
 			(project "DualCore6502Whole"
 				(path "/93e0914e-b2e9-49c2-95f2-7cc419f4ea20/3412cf2c-7ca6-479d-a9c2-89b197305d30"
-					(reference "#PWR119")
+					(reference "#PWR148")
 					(unit 1)
 				)
@@
 		(dnp no)
 		(fields_autoplaced yes)
-		(property "Reference" "#PWR113"
+		(property "Reference" "#PWR142"
 			(at 161.29 83.82 0)
 			(effects
@@
 			(project "DualCore6502Whole"
 				(path "/93e0914e-b2e9-49c2-95f2-7cc419f4ea20/3412cf2c-7ca6-479d-a9c2-89b197305d30"
-					(reference "#PWR113")
+					(reference "#PWR142")
 					(unit 1)
 				)
@@
 		(dnp no)
 		(fields_autoplaced yes)
-		(property "Reference" "U19"
+		(property "Reference" "U22"
 			(at 50.8 171.4499 0)
 			(effects
@@
 			(project ""
 				(path "/93e0914e-b2e9-49c2-95f2-7cc419f4ea20/3412cf2c-7ca6-479d-a9c2-89b197305d30"
-					(reference "U19")
+					(reference "U22")
 					(unit 5)
 				)
@@
 		(dnp no)
 		(fields_autoplaced yes)
-		(property "Reference" "U19"
+		(property "Reference" "U22"
 			(at 77.4617 90.17 0)
 			(effects
@@
 			(project ""
 				(path "/93e0914e-b2e9-49c2-95f2-7cc419f4ea20/3412cf2c-7ca6-479d-a9c2-89b197305d30"
-					(reference "U19")
+					(reference "U22")
 					(unit 2)
 				)
@@
 		(dnp no)
 		(fields_autoplaced yes)
-		(property "Reference" "#PWR110"
+		(property "Reference" "#PWR139"
 			(at 64.77 182.88 0)
 			(effects
@@
 			(project "DualCore6502Whole"
 				(path "/93e0914e-b2e9-49c2-95f2-7cc419f4ea20/3412cf2c-7ca6-479d-a9c2-89b197305d30"
-					(reference "#PWR110")
+					(reference "#PWR139")
 					(unit 1)
 				)
@@
 		(dnp no)
 		(fields_autoplaced yes)
-		(property "Reference" "#PWR109"
+		(property "Reference" "#PWR138"
 			(at 64.77 172.72 0)
 			(effects
@@
 			(project "DualCore6502Whole"
 				(path "/93e0914e-b2e9-49c2-95f2-7cc419f4ea20/3412cf2c-7ca6-479d-a9c2-89b197305d30"
-					(reference "#PWR109")
+					(reference "#PWR138")
 					(unit 1)
 				)
@@
 		(dnp no)
 		(fields_autoplaced yes)
-		(property "Reference" "U19"
+		(property "Reference" "U22"
 			(at 77.4617 109.22 0)
 			(effects
@@
 			(project ""
 				(path "/93e0914e-b2e9-49c2-95f2-7cc419f4ea20/3412cf2c-7ca6-479d-a9c2-89b197305d30"
-					(reference "U19")
+					(reference "U22")
 					(unit 4)
 				)
@@
 		(dnp no)
 		(fields_autoplaced yes)
-		(property "Reference" "#PWR114"
+		(property "Reference" "#PWR143"
 			(at 186.69 81.28 0)
 			(effects
@@
 			(project "DualCore6502Whole"
 				(path "/93e0914e-b2e9-49c2-95f2-7cc419f4ea20/3412cf2c-7ca6-479d-a9c2-89b197305d30"
-					(reference "#PWR114")
+					(reference "#PWR143")
 					(unit 1)
 				)
@@
 		(dnp no)
 		(fields_autoplaced yes)
-		(property "Reference" "#PWR116"
+		(property "Reference" "#PWR145"
 			(at 200.66 81.28 0)
 			(effects
@@
 			(project "DualCore6502Whole"
 				(path "/93e0914e-b2e9-49c2-95f2-7cc419f4ea20/3412cf2c-7ca6-479d-a9c2-89b197305d30"
-					(reference "#PWR116")
+					(reference "#PWR145")
 					(unit 1)
 				)
@@
 		(dnp no)
 		(fields_autoplaced yes)
-		(property "Reference" "#PWR111"
+		(property "Reference" "#PWR140"
 			(at 135.89 81.28 0)
 			(effects
@@
 			(project "DualCore6502Whole"
 				(path "/93e0914e-b2e9-49c2-95f2-7cc419f4ea20/3412cf2c-7ca6-479d-a9c2-89b197305d30"
-					(reference "#PWR111")
+					(reference "#PWR140")
 					(unit 1)
 				)
@@
 		(dnp no)
 		(fields_autoplaced yes)
-		(property "Reference" "#PWR118"
+		(property "Reference" "#PWR147"
 			(at 220.98 81.28 0)
 			(effects
@@
 			(project "DualCore6502Whole"
 				(path "/93e0914e-b2e9-49c2-95f2-7cc419f4ea20/3412cf2c-7ca6-479d-a9c2-89b197305d30"
-					(reference "#PWR118")
+					(reference "#PWR147")
 					(unit 1)
 				)
@@
 		(dnp no)
 		(fields_autoplaced yes)
-		(property "Reference" "#PWR108"
+		(property "Reference" "#PWR136"
 			(at 62.23 78.74 0)
 			(effects
@@
 			(project "DualCore6502Whole"
 				(path "/93e0914e-b2e9-49c2-95f2-7cc419f4ea20/3412cf2c-7ca6-479d-a9c2-89b197305d30"
-					(reference "#PWR108")
+					(reference "#PWR136")
 					(unit 1)
 				)
@@
 		(dnp no)
 		(fields_autoplaced yes)
-		(property "Reference" "#PWR106"
+		(property "Reference" "#PWR134"
 			(at 43.18 163.83 0)
 			(effects
@@
 			(project "DualCore6502Whole"
 				(path "/93e0914e-b2e9-49c2-95f2-7cc419f4ea20/3412cf2c-7ca6-479d-a9c2-89b197305d30"
-					(reference "#PWR106")
+					(reference "#PWR134")
 					(unit 1)
 				)
@@
 		(dnp no)
 		(fields_autoplaced yes)
-		(property "Reference" "#PWR120"
+		(property "Reference" "#PWR137"
 			(at 68.58 120.65 0)
 			(effects
@@
 			(project "DualCore6502Whole"
 				(path "/93e0914e-b2e9-49c2-95f2-7cc419f4ea20/3412cf2c-7ca6-479d-a9c2-89b197305d30"
-					(reference "#PWR120")
+					(reference "#PWR137")
 					(unit 1)
 				)
@@
 		(on_board yes)
 		(dnp no)
-		(property "Reference" "R14"
+		(property "Reference" "R19"
 			(at 233.68 80.0099 0)
 			(effects
@@
 			(project "DualCore6502Whole"
 				(path "/93e0914e-b2e9-49c2-95f2-7cc419f4ea20/3412cf2c-7ca6-479d-a9c2-89b197305d30"
-					(reference "R14")
+					(reference "R19")
 					(unit 1)
 				)
@@
 		(dnp no)
 		(fields_autoplaced yes)
-		(property "Reference" "#PWR117"
+		(property "Reference" "#PWR146"
 			(at 210.82 81.28 0)
 			(effects
@@
 			(project "DualCore6502Whole"
 				(path "/93e0914e-b2e9-49c2-95f2-7cc419f4ea20/3412cf2c-7ca6-479d-a9c2-89b197305d30"
-					(reference "#PWR117")
+					(reference "#PWR146")
 					(unit 1)
 				)
@@
 		(dnp no)
 		(fields_autoplaced yes)
-		(property "Reference" "#PWR115"
+		(property "Reference" "#PWR144"
 			(at 176.53 83.82 0)
 			(effects
@@
 			(project "DualCore6502Whole"
 				(path "/93e0914e-b2e9-49c2-95f2-7cc419f4ea20/3412cf2c-7ca6-479d-a9c2-89b197305d30"
-					(reference "#PWR115")
+					(reference "#PWR144")
 					(unit 1)
 				)
@@
 		(on_board yes)
 		(dnp no)
-		(property "Reference" "R12"
+		(property "Reference" "R17"
 			(at 213.36 80.0099 0)
 			(effects
@@
 			(project "DualCore6502Whole"
 				(path "/93e0914e-b2e9-49c2-95f2-7cc419f4ea20/3412cf2c-7ca6-479d-a9c2-89b197305d30"
-					(reference "R12")
+					(reference "R17")
 					(unit 1)
 				)

Commit message: Basic PCB layout
Parts:
- J6: value Bus 1 -> RCBus; footprint RCBus:RCBus_PinSocket_2x40_P2.54mm_Vertical -> RCBus:RCBus_PinSocket_2x40_P2.54mm_Vertical_DC
- U21: renamed from U22; footprint Package_DIP:DIP-14_W7.62mm -> Package_DIP:DIP-14_W7.62mm_Socket
- renumbered C28 to C27
Connections:
- net CPU1_CLK: now also J6.42 (Pin_42); no longer J6.78 (Pin_78)
- net CPU2_CLK: now also J6.43 (Pin_43); no longer J6.79 (Pin_79)
- net ~{ACIA_CS}: now also J6.79 (Pin_79); no longer J6.42 (Pin_42)
- net ~{IO_4_CS}: now also J6.45 (Pin_45); no longer J6.43 (Pin_43)
- net ~{IO_5_CS}: now also J6.46 (Pin_46); no longer J6.44 (Pin_44)
- net ~{IO_6_CS}: now also J6.47 (Pin_47); no longer J6.45 (Pin_45)
- net ~{IO_7_CS}: now also J6.48 (Pin_48); no longer J6.46 (Pin_46)
- net ~{VIA_CS}: now also J6.78 (Pin_78); no longer J6.41 (Pin_41)
- net TX: now reaches J6.35 (Pin_35)
- net RX: now reaches J6.36 (Pin_36)
- new net MAIN_CLK: J6.41 (Pin_41)
- no-connect marks 27 -> 24
