File: schematics/DualCore6502Whole/tick_timer.kicad_sch (KiCad schematic)
At the start: 9 parts, among them U23 7555, U5 74HC02

Commit message: Basic PCB layout
Parts:
- added TP7: 1KHz, TestPoint:TestPoint_Pad_D1.5mm, symbol Connector:TestPoint
- JP2: value Tick 1 -> NMI1; footprint Jumper:SolderJumper-2_P1.3mm_Bridged_RoundedPad1.0x1.5mm -> Connector_PinHeader_2.54mm:PinHeader_1x02_P2.54mm_Vertical
- JP3: value Tick 2 -> NMI2; footprint Jumper:SolderJumper-2_P1.3mm_Bridged_RoundedPad1.0x1.5mm -> Connector_PinHeader_2.54mm:PinHeader_1x02_P2.54mm_Vertical
- U22: renamed from U23; footprint Package_DIP:DIP-8_W7.62mm -> Package_DIP:DIP-8_W7.62mm_Socket
- U4: renamed from U5; footprint Package_DIP:DIP-14_W7.62mm -> Package_DIP:DIP-14_W7.62mm_Socket
- renumbered C29 to C28, C30 to C29
Connections:
- net at U22.3 (Q), U4.11, U4.9: now also TP7.1
Changed lines of the file:
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@@
+	)
+	(junction
+		(at 139.7 86.36)
+		(diameter 0)
+		(color 0 0 0 0)
 	)
 	(junction
@@
 	(wire
 		(pts
-			(xy 119.38 86.36) (xy 149.86 86.36)
+			(xy 119.38 86.36) (xy 139.7 86.36)
 		)
 		(stroke
@@
 	(wire
 		(pts
+			(xy 139.7 86.36) (xy 149.86 86.36)
+		)
+		(stroke
+			(width 0)
+			(type default)
+		)
+	)
+	(wire
+		(pts
 			(xy 81.28 116.84) (xy 123.19 116.84)
 		)
@@
 		(pts
 			(xy 149.86 86.36) (xy 149.86 113.03)
+		)
+		(stroke
+			(width 0)
+			(type default)
+		)
+	)
+	(wire
+		(pts
+			(xy 139.7 82.55) (xy 139.7 86.36)
 		)
 		(stroke
@@
 	(text "Invert so ~{CPUn_NMI} is pulled high during reset."
 		(exclude_from_sim no)
-		(at 163.83 74.168 0)
+		(at 174.244 75.438 0)
 		(effects
 			(font
@@
 		(dnp no)
 		(fields_autoplaced yes)
-		(property "Reference" "U5"
+		(property "Reference" "U4"
 			(at 163.83 101.6 0)
 			(effects
@@
 			)
 		)
-		(property "Footprint" "Package_DIP:DIP-14_W7.62mm"
+		(property "Footprint" "Package_DIP:DIP-14_W7.62mm_Socket"
 			(at 163.83 110.49 0)
 			(effects
@@
 			(project "DualCore6502Whole"
 				(path "/93e0914e-b2e9-49c2-95f2-7cc419f4ea20/731fd70c-eedb-4909-a6f7-e3ec3269813b"
-					(reference "U5")
+					(reference "U4")
 					(unit 3)
 				)
@@
 		(dnp no)
 		(fields_autoplaced yes)
-		(property "Reference" "#PWR150"
+		(property "Reference" "#PWR146"
 			(at 106.68 114.3 0)
 			(effects
@@
 			(project "DualCore6502Whole"
 				(path "/93e0914e-b2e9-49c2-95f2-7cc419f4ea20/731fd70c-eedb-4909-a6f7-e3ec3269813b"
-					(reference "#PWR150")
+					(reference "#PWR146")
 					(unit 1)
 				)
@@
 		(dnp no)
 		(fields_autoplaced yes)
-		(property "Reference" "#PWR149"
+		(property "Reference" "#PWR145"
 			(at 106.68 78.74 0)
 			(effects
@@
 			(project "DualCore6502Whole"
 				(path "/93e0914e-b2e9-49c2-95f2-7cc419f4ea20/731fd70c-eedb-4909-a6f7-e3ec3269813b"
-					(reference "#PWR149")
+					(reference "#PWR145")
 					(unit 1)
 				)
@@
 			)
 		)
-		(property "Value" "Tick 2"
+		(property "Value" "NMI2"
 			(at 181.61 107.95 0)
 			(effects
@@
 			)
 		)
-		(property "Footprint" "Jumper:SolderJumper-2_P1.3mm_Bridged_RoundedPad1.0x1.5mm"
+		(property "Footprint" "Connector_PinHeader_2.54mm:PinHeader_1x02_P2.54mm_Vertical"
 			(at 181.61 110.49 0)
 			(effects
@@
 				(path "/93e0914e-b2e9-49c2-95f2-7cc419f4ea20/731fd70c-eedb-4909-a6f7-e3ec3269813b"
 					(reference "JP3")
+					(unit 1)
+				)
+			)
+		)
+	)
+	(symbol
+		(lib_id "Connector:TestPoint")
+		(at 139.7 82.55 0)
+		(unit 1)
+		(exclude_from_sim no)
+		(in_bom yes)
+		(on_board yes)
+		(dnp no)
+		(fields_autoplaced yes)
+		(property "Reference" "TP7"
+			(at 142.24 77.9779 0)
+			(effects
+				(font
+					(size 1.27 1.27)
+				)
+				(justify left)
+			)
+		)
+		(property "Value" "1KHz"
+			(at 142.24 80.5179 0)
+			(effects
+				(font
+					(size 1.27 1.27)
+				)
+				(justify left)
+			)
+		)
+		(property "Footprint" "TestPoint:TestPoint_Pad_D1.5mm"
+			(at 144.78 82.55 0)
+			(effects
+				(font
+					(size 1.27 1.27)
+				)
+				(hide yes)
+			)
+		)
+		(property "Datasheet" "~"
+			(at 144.78 82.55 0)
+			(effects
+				(font
+					(size 1.27 1.27)
+				)
+				(hide yes)
+			)
+		)
+		(property "Description" "test point"
+			(at 139.7 82.55 0)
+			(effects
+				(font
+					(size 1.27 1.27)
+				)
+				(hide yes)
+			)
+		)
+		(pin "1"
+		)
+		(instances
+			(project ""
+				(path "/93e0914e-b2e9-49c2-95f2-7cc419f4ea20/731fd70c-eedb-4909-a6f7-e3ec3269813b"
+					(reference "TP7")
 					(unit 1)
 				)
@@
 		(dnp no)
 		(fields_autoplaced yes)
-		(property "Reference" "U5"
+		(property "Reference" "U4"
 			(at 163.83 80.01 0)
 			(effects
@@
 			)
 		)
-		(property "Footprint" "Package_DIP:DIP-14_W7.62mm"
+		(property "Footprint" "Package_DIP:DIP-14_W7.62mm_Socket"
 			(at 163.83 88.9 0)
 			(effects
@@
 			(project "DualCore6502Whole"
 				(path "/93e0914e-b2e9-49c2-95f2-7cc419f4ea20/731fd70c-eedb-4909-a6f7-e3ec3269813b"
-					(reference "U5")
+					(reference "U4")
 					(unit 4)
 				)
@@
 		(on_board yes)
 		(dnp no)
-		(property "Reference" "U23"
+		(property "Reference" "U22"
 			(at 108.8741 78.74 0)
 			(effects
@@
 			)
 		)
-		(property "Footprint" "Package_DIP:DIP-8_W7.62mm"
+		(property "Footprint" "Package_DIP:DIP-8_W7.62mm_Socket"
 			(at 123.19 101.6 0)
 			(effects
@@
 			(project "DualCore6502Whole"
 				(path "/93e0914e-b2e9-49c2-95f2-7cc419f4ea20/731fd70c-eedb-4909-a6f7-e3ec3269813b"
-					(reference "U23")
+					(reference "U22")
 					(unit 1)
 				)
@@
 			)
 		)
-		(property "Value" "Tick 1"
+		(property "Value" "NMI1"
 			(at 181.61 86.36 0)
 			(effects
@@
 			)
 		)
-		(property "Footprint" "Jumper:SolderJumper-2_P1.3mm_Bridged_RoundedPad1.0x1.5mm"
+		(property "Footprint" "Connector_PinHeader_2.54mm:PinHeader_1x02_P2.54mm_Vertical"
 			(at 181.61 88.9 0)
 			(effects
@@
 		(dnp no)
 		(fields_autoplaced yes)
-		(property "Reference" "#PWR148"
+		(property "Reference" "#PWR144"
 			(at 88.9 114.3 0)
 			(effects
@@
 			(project "DualCore6502Whole"
 				(path "/93e0914e-b2e9-49c2-95f2-7cc419f4ea20/731fd70c-eedb-4909-a6f7-e3ec3269813b"
-					(reference "#PWR148")
+					(reference "#PWR144")
 					(unit 1)
 				)
@@
 		(dnp no)
 		(fields_autoplaced yes)
-		(property "Reference" "#PWR152"
+		(property "Reference" "#PWR148"
 			(at 128.27 78.74 0)
 			(effects
@@
 			(project "DualCore6502Whole"
 				(path "/93e0914e-b2e9-49c2-95f2-7cc419f4ea20/731fd70c-eedb-4909-a6f7-e3ec3269813b"
-					(reference "#PWR152")
+					(reference "#PWR148")
 					(unit 1)
 				)
@@
 		(dnp no)
 		(fields_autoplaced yes)
-		(property "Reference" "C29"
+		(property "Reference" "C28"
 			(at 92.71 102.8699 0)
 			(effects
@@
 			(project "DualCore6502Whole"
 				(path "/93e0914e-b2e9-49c2-95f2-7cc419f4ea20/731fd70c-eedb-4909-a6f7-e3ec3269813b"
-					(reference "C29")
+					(reference "C28")
 					(unit 1)
 				)
@@
 		(dnp no)
 		(fields_autoplaced yes)
-		(property "Reference" "C30"
+		(property "Reference" "C29"
 			(at 127 121.9199 0)
 			(effects
@@
 			(project "DualCore6502Whole"
 				(path "/93e0914e-b2e9-49c2-95f2-7cc419f4ea20/731fd70c-eedb-4909-a6f7-e3ec3269813b"
-					(reference "C30")
+					(reference "C29")
 					(unit 1)
 				)
@@
 		(dnp no)
 		(fields_autoplaced yes)
-		(property "Reference" "#PWR151"
+		(property "Reference" "#PWR147"
 			(at 123.19 133.35 0)
 			(effects
@@
 			(project "DualCore6502Whole"
 				(path "/93e0914e-b2e9-49c2-95f2-7cc419f4ea20/731fd70c-eedb-4909-a6f7-e3ec3269813b"
-					(reference "#PWR151")
+					(reference "#PWR147")
 					(unit 1)
 				)
@@
 		(dnp no)
 		(fields_autoplaced yes)
-		(property "Reference" "#PWR153"
+		(property "Reference" "#PWR149"
 			(at 152.4 121.92 0)
 			(effects
@@
 			(project "DualCore6502Whole"
 				(path "/93e0914e-b2e9-49c2-95f2-7cc419f4ea20/731fd70c-eedb-4909-a6f7-e3ec3269813b"
-					(reference "#PWR153")
+					(reference "#PWR149")
 					(unit 1)
 				)
